File: Music-player.kicad_sch (KiCad schematic)
At the start: 28 parts, among them J1 USB_C_Receptacle_USB2.0_14P, SW1 RESET, U1 TVS1400DRV, U2 nRF5340-QKxx, U3 NCP1117-3.3_SOT223, Y1 SG-3030CM, Y2 32MHz

Commit message: Add files via upload
Parts:
- removed AE1: Antenna_Chip, symbol Device:Antenna_Chip
- removed C8: 100n, symbol Device:C
- removed L4: 10uH, symbol Device:L
- removed Y1: SG-3030CM, Oscillator:Oscillator_SMD_SeikoEpson_SG3030CM, symbol Oscillator:SG-3030CM
- added C14: 0.7p, symbol Device:C
- added C15: NC, symbol Device:C
- added C16, C17, C18, C19, C20, C21, C22, C23, C24, C25, C26, C27, C28: 100n, symbol Device:C
- added C29: 4.7u, symbol Device:C
- added D1: POWER, symbol Device:LED
- added D2: IO_STATUS, symbol Device:LED
- added D3: POWER STATUS, symbol Device:LED
- added D5: LED, symbol Device:LED
- added J2: Screw_Terminal_01x04, symbol Connector:Screw_Terminal_01x04
- added J3: Screw_Terminal_01x02, symbol Connector:Screw_Terminal_01x02
- added L5: 2.2n, symbol Device:L
- added Q1, Q2: DMG2301L, Package_TO_SOT_SMD:SOT-23, symbol Transistor_FET:DMG2301L
- added R10: 2k, symbol Device:R
- added R12: 470, symbol Device:R
- added R4: 2R2, symbol Device:R
- added R5, R7: 100, symbol Device:R
- added R6: 33, symbol Device:R
- added R8, R9: 1M, symbol Device:R
- added U5: MCP73831-2-OT, Package_TO_SOT_SMD:SOT-23-5, symbol Battery_Management:MCP73831-2-OT
- added Y1: MU00525-32-768K, symbol Device:Crystal_Small
- C12: value 100nF -> 1u
- C13: value 100NF -> 2.2n
- C9: value 1u -> 4.7u
- L2, L3: value 10uH -> 10u
Connections:
- net +3V3: now also U2.A21 (DCC), U2.B10 (DCCD), C16.1, C17.1, C18.1, C19.1, C20.1, C21.1, C22.1, C23.1, C24.1, C25.1, C26.1, C27.1, C28.1, J2.2 (Pin_2); no longer R3.1
- net GND: now also C14.2, C15.2, C16.2, C17.2, C18.2, C19.2, C20.2, C21.2, C22.2, C23.2, C24.2, C25.2, C26.2, C27.2, C28.2, C29.2, D1.1 (K), D2.1 (K), D3.1 (K), J2.1 (Pin_1), J3.1 (Pin_1), R10.2, R9.2, U5.2 (V_{SS}); no longer U2.AA1 (NFC2/P0.03), U2.W1 (NFC1/P0.02)
- net USB_POWER: now also Q1.1 (G), Q2.3 (D), R4.1; no longer J1.A4 (VBUS), J1.A9 (VBUS), J1.B4 (VBUS), J1.B9 (VBUS), U2.A5 (VBUS)
- net XL1: now also Y1.2
- net at C13.1, U2.G31 (DECRF): now also C12.1, L3.1, U2.A27 (DECR)
- net at C10.1, U2.A15 (DECD): now also L2.1; no longer L3.1
- net at L1.2, U2.J1 (DCCH): no longer C11.1
- net at R3.2, SW1.2: no longer U2.AC31 (~{RESET})
- net at U2.L31 (ANT): now also C14.1, L5.2
- net IO1: now reaches U2.M2 (P1.00)
- net IO1: now also R6.1
- net IO2: now reaches U2.P2 (P1.01)
- net IO2: now also R7.1
- net XL2: now reaches U2.R1 (XL2/P0.01)
- net XL2: now also Y1.1
- net AIN0: now reaches U2.V2 (AIN0/P0.04)
- net AIN0: now also R8.2, R9.1
- net J-LINK2 renamed SWDIO
- net SWDIO: now also J2.4 (Pin_4)
- net J-LINK4 renamed SWDCLK
- net SWDCLK: now also J2.3 (Pin_3)
- new net: C9.1, R4.2, U2.A5 (VBUS)
- new net: D1.2 (A), R5.2
- new net: D2.2 (A), R6.2
- new net: D5.1 (K), R12.1
- new net: R12.2, U5.1 (STAT)
- new net: R10.1, U5.5 (PROG)
- new net: D3.2 (A), R7.2
- new net 3V3: R5.1
- new net CHARGING: C29.1, D5.2 (A), J1.A4 (VBUS), J1.A9 (VBUS), J1.B4 (VBUS), J1.B9 (VBUS), Q2.2 (S), U5.4 (V_{DD})
- new net LI_ION: C11.1, J3.2 (Pin_2), Q1.2 (S), U5.3 (V_{BAT})
- new net RESET: R3.1, U2.AC31 (~{RESET})
- new net RF: C15.1, L5.1
- new net VBAT: Q1.3 (D), Q2.1 (G), R8.1
- no-connect marks 1 -> 0
Other:
- note added: "BATTERY TERMINAL"
- note added: "CHARGING CIRCUIT"
- note added: "CRYSTAL"
- note added: "CRYSTAL MODULE"
- note added: "J-LINK CONNECTOR"
- note added: "REC. CL {6pF, 7pF, 9pF}"
- note added: "RESET"
- note added: "STATUS LED"
- note added: "USE INTERNAL CAPACITOR (6 pF) VALUE C6PF (1) PAGE 101"
- note added: "VDD 100NF"
- note added: "VOLTAGE DIVIDER"
- moved on the sheet: C1, C10, C12, C13, C2, C3, C5, C6, C7, J1, R1, R2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

Commit message: Add files via upload
Parts:
- added C30, C31, C32, C33, C34, C35, C36, C38: 100n, symbol Device:C
- added C37: 10u, symbol Device:C
- added C8: 1u, symbol Device:C
- added FB1, FB2: BLM18PG221SN1D, symbol Device:FerriteBead
- added J4: MSD-4-A, MSD-4-A:CUI_MSD-4-A, symbol My-Kicad-Library:MSD-4-A
- added J5: SJ-43514, SJ-43514:CUI_SJ-43514, symbol My-Kicad-Library:SJ-43514
- added R11: NC, symbol Device:R
- added R13, R14: 10K, symbol Device:R
- added SW2: PLAY/STOP, symbol Switch:SW_Push
- added SW3: SKIP, symbol Switch:SW_Push
- added SW4: EXIT, symbol Switch:SW_Push
- added SW5: OPTIONS, symbol Switch:SW_Push
- added SW6: EC11_L, symbol Device:RotaryEncoder_Switch
- added SW7: POWER, symbol Switch:SW_Push
- added U4: (no value), symbol My-Kicad-Library:ST7789
- added U6: TPA6132A2RTE, Package_DFN_QFN:WQFN-16-1EP_3x3mm_P0.5mm_EP1.6x1.6mm_ThermalVias, symbol Amplifier_Audio:TPA6132A2RTE
- added U7: PCM5102A, Package_SO:TSSOP-20_4.4x6.5mm_P0.65mm, symbol Audio:PCM5102A
- C24, C25: value 100n -> 1u
- C26: value 100n -> 2.2u
- C27: value 100n -> 4.7u
- C29: value 4.7u -> 100n
- C3: value 1u -> 100n
- C5: value 1u -> 4.7u
- C6: value 12pF -> 4.7u
- C7: value 12pF -> 100n
- Y2: value 32MHz -> MU00525-32-768K
Connections:
- net VBAT is gone; now on net USB_POWER: Q1.3 (D), Q2.1 (G), R8.1
- net +3V3: now also C29.1, C30.1, C31.1, C32.1, C33.1, C34.1, C35.1, C36.1, C37.1, C38.1; no longer C2.1, J2.2 (Pin_2), L1.1, L2.2, L3.2, U2.A19 (VDD), U2.A21 (DCC), U2.AC1 (VDD), U2.AG1 (VDD), U2.AJ31 (VDD), U2.AL11 (VDD), U2.AL17 (VDD), U2.AL25 (VDD), U2.AL3 (VDD), U2.AL7 (VDD), U2.B10 (DCCD), U2.B28 (VDD), U2.B8 (VDD), U2.C1 (VDD), U2.E1 (VDDH), U2.E31 (VDD), U2.L1 (VDD), U2.N31 (VDD), U2.U1 (VDD), U3.2 (VO)
- net CHARGING: now also C6.1; no longer C29.1
- net GND: now also C30.2, C31.2, C32.2, C33.2, C34.2, C35.2, C36.2, C37.2, C38.2, C8.2, FB2.1, J4.6 (VSS), J4.G1 (COVER_GND), J4.G2 (COVER_GND__1), J4.G3 (COVER_GND__2), J4.G4 (COVER_GND__3), SW2.2, SW3.2, SW4.2, SW5.2, SW6.C, SW6.S2, SW7.2, U4.1 (GND), U7.19 (DGND)
- net XC1: no longer C6.1
- net XC2: no longer C7.1
- net CD: now reaches U2.AA1 (NFC2/P0.03)
- net CD: now also J4.CD, R13.1
- net MSD_CS: now reaches U2.AE1 (TWI/P1.02)
- net MSD_CS: now also J4.2 (CS)
- net SCK: now reaches U2.AH2 (SCK/TRACEDATA3/P0.08)
- net SCK: now also J4.5 (SCK), U4.3 (SCL)
- net MOSI: now reaches U2.AJ1 (MOSI/TRACEDATA2/P0.09)
- net MOSI: now also J4.3 (MOSI), U4.4 (SDA)
- net PLAY/STOP: now reaches U2.AK16 (P0.20)
- net PLAY/STOP: now also SW2.1
- net SKIP: now reaches U2.AK18 (P0.22)
- net SKIP: now also SW3.1
- net MISO: now reaches U2.AK2 (MISO/TRACEDATA1/P0.10)
- net MISO: now also J4.7 (MISO), R14.1
- net EXIT: now reaches U2.AK20 (P0.23)
- net EXIT: now also SW4.1
- net OPTIONS: now reaches U2.AK22 (P1.05)
- net OPTIONS: now also SW5.1
- net EC11_B: now reaches U2.AK26 (P1.09)
- net EC11_B: now also SW6.B
- net EC11_A: now reaches U2.AK28 (AIN4/P0.25)
- net EC11_A: now also SW6.A
- net SELECT: now reaches U2.AK30 (AIN6/P0.27)
- net SELECT: now also SW6.S1
- net POWER: now reaches U2.AK6 (DCX/TRACECLK/P0.12)
- net POWER: now also R11.1
- net RES: now reaches U2.AL19 (P1.04)
- net RES: now also U4.5 (RES)
- net DC: now reaches U2.AL21 (P1.06)
- net DC: now also U4.6 (DC)
- net SST_CS: now reaches U2.AL23 (P1.08)
- net SST_CS: now also U4.7 (CS)
- net BLK: now reaches U2.AL27 (P0.24)
- net BLK: now also U4.8 (BLK)
- net 3V3 renamed VDD
- net VDD: now also C2.1, J2.2 (Pin_2), L1.1, L2.2, L3.2, U2.A19 (VDD), U2.A21 (DCC), U2.AC1 (VDD), U2.AG1 (VDD), U2.AJ31 (VDD), U2.AL11 (VDD), U2.AL17 (VDD), U2.AL25 (VDD), U2.AL3 (VDD), U2.AL7 (VDD), U2.B10 (DCCD), U2.B28 (VDD), U2.B8 (VDD), U2.C1 (VDD), U2.E1 (VDDH), U2.E31 (VDD), U2.L1 (VDD), U2.N31 (VDD), U2.U1 (VDD), U3.2 (VO), FB1.1, J4.4 (VCC), R13.2, R14.2, U4.2 (VCC)
- new net: R11.2, SW7.1
- new net GNDA: FB2.2, U7.9 (AGND)
- new net RING_1: J5.3
- new net RING_2: J5.4
- new net SLEEVE: J5.1
- new net TIP: J5.2
- new net VDDA: C7.1, C8.1, FB1.2
- no-connect marks 0 -> 3
Other:
- note added: "BUTTONS"
- note added: "C16-C23 VDD"
- note added: "C24 A19"
- note added: "C25 B8"
- note added: "C26 L1"
- note added: "C27 E1"
- note added: "C28 SST7789"
- note added: "C29-32 BUTTONS"
- note added: "C33 EC11 SELECT"
- note added: "C34 EC11_A"
- note added: "C35 EC11_B"
- note added: "C36 MSD_4_A"
- note added: "C37-C38 MSD-4-A"
- note added: "CRYSTALS"
- note added: "CS MUST HAVE INT RESISTOR ENABLED"
- note added: "ENCODER"
- note added: "FINISH THE PCM5102A, TPA6132A2RTE, SJ43514, GND AND VDD SEPERATION, ANTENNA"
- note added: "HEADERS"
- note added: "SST7789"
- note added: "USE 6pF INT CAP"
- note removed: "CRYSTAL"
- note removed: "CRYSTAL MODULE"
- note removed: "REC. CL {6pF, 7pF, 9pF}"
- note removed: "VDD 100NF"
- moved on the sheet: C1, C16, C17, C18, C19, C2, C20, C21, C22, C23, C24, C25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

Commit message: Add files via upload
Parts:
- removed U6: TPA6132A2RTE, Package_DFN_QFN:WQFN-16-1EP_3x3mm_P0.5mm_EP1.6x1.6mm_ThermalVias, symbol Amplifier_Audio:TPA6132A2RTE
- removed U7: PCM5102A, Package_SO:TSSOP-20_4.4x6.5mm_P0.65mm, symbol Audio:PCM5102A
- added C39, C40, C41, C43, C44, C45, C46, C50, C53: 1u, symbol Device:C
- added C42, C48, C51, C52: 100n, symbol Device:C
- added C47: 2.2u, symbol Device:C
- added C49: 10u, symbol Device:C
- added U6: TPA6132A2RTE, Package_DFN_QFN:WQFN-16-1EP_3x3mm_P0.5mm_EP1.6x1.6mm_ThermalVias, symbol My-Kicad-Library:TPA6132A2RTE
- added U8: PCM5102A, Package_SO:TSSOP-20_4.4x6.5mm_P0.65mm, symbol My-Kicad-Library:PCM5102A
- Y2: value MU00525-32-768K -> ECS-320-8-37B-CKY-TR
Connections:
- net +3V3 is gone; now on net VDD: C16.1, C17.1, C18.1, C19.1, C20.1, C21.1, C22.1, C23.1, C24.1, C25.1, C26.1, C27.1, C28.1, C29.1, C30.1, C31.1, C32.1, C33.1, C34.1, C35.1, C36.1, C37.1, C38.1
- net SLEEVE is gone; now on net GNDA: J5.1
- net GND: now also C52.2, C53.2, U8.10 (DEMP), U8.11 (FLT), U8.16 (FMT), U8.19 (DGND)
- net GNDA: now also C40.2, C41.2, C42.2, C46.2, C47.2, C48.2, C49.2, C50.2, C51.2, U6.10 (PGND), U6.15 (SGND), U6.17 (EP), U6.2 (INL+), U6.3 (INR+), U8.3 (CPGND), U8.9 (AGND)
- net RING_1: now also U6.5 (OUTR)
- net TIP: now also U6.16 (OUTL)
- net VDD: now also C52.1, C53.1, U8.20 (DVDD)
- net VDDA: now also C42.1, C48.1, C49.1, C50.1, C51.1, U6.14 (VDD), U8.1 (CPVDD), U8.8 (AVDD)
- net G1: now reaches U2.A17 (P1.13)
- net G1: now also U6.7 (G1)
- net LRCK: now reaches U2.B14 (P1.15)
- net LRCK: now also U8.15 (LRCK)
- net DIN: now reaches U2.B16 (P1.14)
- net DIN: now also U8.14 (DIN)
- net BCK: now reaches U2.B18 (P1.12)
- net BCK: now also U8.13 (BCK)
- net MUTE: now reaches U2.B20 (P1.11)
- net MUTE: now also U8.17 (XSMT)
- net TPA_EN: now reaches U2.B22 (P0.31)
- net TPA_EN: now also U6.13 (EN)
- net G0: now reaches U2.B24 (P0.30)
- net G0: now also U6.6 (G0)
- net RING_2: no longer names the net of J5.4
- new net: C41.1, U8.18 (LDOO)
- new net: C46.1, U6.8 (HPVSS)
- new net: C45.1, U6.11 (CPP)
- new net: C47.1, U6.12 (HPVDD)
- new net: C45.2, U6.9 (CPN)
- new net: C40.1, U8.5 (VNEG)
- new net: C39.1, U8.2 (CAPP)
- new net: C39.2, U8.4 (CAPM)
- new net OUTL: C44.2, U6.1 (INL-)
- new net OUTR: C43.2, U6.4 (INR-)
- new net PCM_OUTL: C44.1, U8.6 (OUTL)
- new net PCM_OUTR: C43.1, U8.7 (OUTR)
- no-connect marks 3 -> 11
Other:
- note added: "C42 PCM5102A PLACE CAREFULLY FOR CPGND"
- note added: "C48-49 PCM"
- note added: "C50-51 TPA"
- note added: "C52-53 PCM"
- note added: "CAPACITORS"
- note added: "CHECK EXACT SPEC LATER"
- note added: "DISABLE NFC IN FIRMWARE"
- note added: "HEADPHONE JACK"
- note added: "MICROSD SOCKET"
- note added: "PCM5102A"
- note added: "SERIES CAPACITOR PLACE CLOSE TO PCM OUTPUT"
- note added: "TPA6132A2RTE"
- moved on the sheet: J4, J5, R13, R14

Commit message: Add files via upload
Parts:
- removed Q1: DMG2301L, Package_TO_SOT_SMD:SOT-23, symbol Transistor_FET:DMG2301L
- added E1: 2450AT18B100E, MyFootprintLibrary:XDCR_2450AT18B100E, symbol My-Kicad-Library:2450AT18B100E
- C1, C10, C11, C12, C13, C14, C15, C16, C17, C18, C19, C2, C20, C21, C22, C23, C24, C25, C26, C27, C28, C29, C3, C30, C31, C32, C33, C34, C35, C36, C37, C38, C39, C4, C40, C41, C42, C43, C44, C45, C46, C47, C48, C49, C5, C50, C51, C52, C53, C6, C7, C8, C9: footprint (none) -> Capacitor_SMD:C_0603_1608Metric
- D1, D2, D3: footprint (none) -> LED_SMD:LED_0603_1608Metric
- D4: renamed from D5; footprint (none) -> LED_SMD:LED_0603_1608Metric
- FB1, FB2, R1, R10, R12, R13, R14, R2, R3, R4, R5, R6, R7, R8, R9: footprint (none) -> Resistor_SMD:R_0603_1608Metric
- J1: footprint (none) -> Connector_USB:USB_C_Receptacle_GCT_USB4105-xx-A_16P_TopMnt_Horizontal
- J2: footprint (none) -> TerminalBlock_Phoenix:TerminalBlock_Phoenix_PT-1,5-4-3.5-H_1x04_P3.50mm_Horizontal
- J3: footprint (none) -> Connector_JST:JST_PH_S2B-PH-K_1x02_P2.00mm_Horizontal
- J4: footprint MSD-4-A:CUI_MSD-4-A -> MyFootprintLibrary:CUI_MSD-4-A
- J5: footprint SJ-43514:CUI_SJ-43514 -> MyFootprintLibrary:SJ-43514_CUD
- L1, L2, L3: footprint (none) -> Inductor_SMD:L_0201_0603Metric
- L5: footprint (none) -> Inductor_SMD:L_0402_1005Metric
- R11: footprint (none) -> Resistor_SMD:R_0603_1608Metric; now not fitted
- SW1, SW2, SW3, SW4, SW5, SW7: footprint (none) -> MyFootprintLibrary:SW_K2-1107ST-A4DW-06_HRO
- SW6: footprint (none) -> Rotary_Encoder:RotaryEncoder_Alps_EC11E-Switch_Vertical_H20mm_MountingHoles
- U4: footprint (none) -> Connector_PinHeader_2.54mm:PinHeader_1x08_P2.54mm_Vertical
- Y1: footprint (none) -> Crystal:Crystal_SMD_3215-2Pin_3.2x1.5mm
- Y2: footprint (none) -> Crystal:Crystal_SMD_3225-4Pin_3.2x2.5mm
Connections:
- net LI_ION: now also R8.1; no longer C11.1, J3.2 (Pin_2), U5.3 (V_{BAT})
- net RF: now also E1.1
- net USB_POWER: now also C11.1, J3.2 (Pin_2), U5.3 (V_{BAT}); no longer R8.1
- no-connect marks 11 -> 20
Other:
- note added: "Bourns SRR1005-100Y"
- note added: "MICROSD SOCKET MSD-4-A"
- note added: "R ON SPI LINE FOR RINGING?"
- note added: "SST7789 SCREEN"
- note added: "muRata LQG15HS2N2B02D"
- note removed: "CHECK EXACT SPEC LATER"
- note removed: "MICROSD SOCKET"
- note removed: "SST7789"
- moved on the sheet: FB2

Commit message: Add files via upload
Parts:
- removed FB2: BLM18PG221SN1D, Resistor_SMD:R_0603_1608Metric, symbol Device:FerriteBead
Connections:
- net LI_ION is gone; now on net USB_POWER: R8.1
Changed lines of the file:
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@@
 		)
 	)
-	(label "LI_ION"
+	(label "VBAT"
 		(at 388.62 20.32 0)
 		(effects
@@
 	)
 	(symbol
-		(lib_id "power:GND")
-		(at 250.19 55.88 0)
-		(unit 1)
-		(body_style 1)
-		(exclude_from_sim no)
-		(in_bom yes)
-		(on_board yes)
-		(in_pos_files yes)
-		(dnp no)
-		(fields_autoplaced yes)
-		(property "Reference" "#PWR033"
-			(at 250.19 62.23 0)
-			(hide yes)
-			(show_name no)
-			(do_not_autoplace no)
-			(effects
-				(font
-					(size 1.27 1.27)
-				)
-			)
-		)
-		(property "Value" "GND"
-			(at 250.19 60.96 0)
-			(show_name no)
-			(do_not_autoplace no)
-			(effects
-				(font
-					(size 1.27 1.27)
-				)
-			)
-		)
-		(property "Footprint" ""
-			(at 250.19 55.88 0)
-			(hide yes)
-			(show_name no)
-			(do_not_autoplace no)
-			(effects
-				(font
-					(size 1.27 1.27)
-				)
-			)
-		)
-		(property "Datasheet" ""
-			(at 250.19 55.88 0)
-			(hide yes)
-			(show_name no)
-			(do_not_autoplace no)
-			(effects
-				(font
-					(size 1.27 1.27)
-				)
-			)
-		)
-		(property "Description" "Power symbol creates a global label with name \"GND\" , ground"
-			(at 250.19 55.88 0)
-			(hide yes)
-			(show_name no)
-			(do_not_autoplace no)
-			(effects
-				(font
-					(size 1.27 1.27)
-				)
-			)
-		)
-		(pin "1"
-		)
-		(instances
-			(project "Music-player"
-				(path "/f98d3056-e9c6-4dc5-a080-338d8b2650d2"
-					(reference "#PWR033")
-					(unit 1)
-				)
-			)
-		)
-	)
-	(symbol
 		(lib_id "Switch:SW_Push")
 		(at 294.64 143.51 0)
@@
 	)
 	(symbol
-		(lib_id "Device:FerriteBead")
-		(at 254 55.88 90)
-		(unit 1)
-		(body_style 1)
-		(exclude_from_sim no)
-		(in_bom yes)
-		(on_board yes)
-		(in_pos_files yes)
-		(dnp no)
-		(property "Reference" "FB2"
-			(at 254 50.038 90)
-			(show_name no)
-			(do_not_autoplace no)
-			(effects
-				(font
-					(size 1.27 1.27)
-				)
-			)
-		)
-		(property "Value" "BLM18PG221SN1D"
-			(at 254 52.07 90)
-			(show_name no)
-			(do_not_autoplace no)
-			(effects
-				(font
-					(size 1.27 1.27)
-				)
-			)
-		)
-		(property "Footprint" "Resistor_SMD:R_0603_1608Metric"
-			(at 254 57.658 90)
-			(hide yes)
-			(show_name no)
-			(do_not_autoplace no)
-			(effects
-				(font
-					(size 1.27 1.27)
-				)
-			)
-		)
-		(property "Datasheet" ""
-			(at 254 55.88 0)
-			(hide yes)
-			(show_name no)
-			(do_not_autoplace no)
-			(effects
-				(font
-					(size 1.27 1.27)
-				)
-			)
-		)
-		(property "Description" "Ferrite bead"
-			(at 254 55.88 0)
-			(hide yes)
-			(show_name no)
-			(do_not_autoplace no)
-			(effects
-				(font
-					(size 1.27 1.27)
-				)
-			)
-		)
-		(pin "1"
-		)
-		(pin "2"
-		)
-		(instances
-			(project "Music-player"
-				(path "/f98d3056-e9c6-4dc5-a080-338d8b2650d2"
-					(reference "FB2")
-					(unit 1)
-				)
-			)
-		)
-	)
-	(symbol
 		(lib_id "My-Kicad-Library:PCM5102A")
 		(at 233.68 245.11 0)
@@
 					(unit 1)
 				)
-			)
-		)
-	)
-	(symbol
-		(lib_id "power:GNDA")
-		(at 257.81 55.88 0)
-		(unit 1)
-		(body_style 1)
-		(exclude_from_sim no)
-		(in_bom yes)
-		(on_board yes)
-		(in_pos_files yes)
-		(dnp no)
-		(fields_autoplaced yes)
-		(property "Reference" "#PWR034"
-			(at 257.81 62.23 0)
-			(hide yes)
-			(show_name no)
-			(do_not_autoplace no)
-			(effects
-				(font
-					(size 1.27 1.27)
-				)
-			)
-		)
-		(property "Value" "GNDA"
-			(at 257.81 60.96 0)
-			(show_name no)
-			(do_not_autoplace no)
-			(effects
-				(font
-					(size 1.27 1.27)
-				)
-			)
-		)
-		(property "Footprint" ""
-			(at 257.81 55.88 0)
-			(hide yes)
-			(show_name no)
-			(do_not_autoplace no)
-			(effects
-				(font
-					(size 1.27 1.27)
-				)
-			)
-		)
-		(property "Datasheet" ""
-			(at 257.81 55.88 0)
-			(hide yes)
-			(show_name no)
-			(do_not_autoplace no)
-			(effects
-				(font
-					(size 1.27 1.27)
-				)
-			)
-		)
-		(property "Description" "Power symbol creates a global label with name \"GNDA\" , analog ground"
-			(at 257.81 55.88 0)
-			(hide yes)
-			(show_name no)
-			(do_not_autoplace no)
-			(effects
-				(font
-					(size 1.27 1.27)
-				)
-			)
-		)
-		(pin "1"
-		)
-		(instances
-			(project "Music-player"
-				(path "/f98d3056-e9c6-4dc5-a080-338d8b2650d2"
-					(reference "#PWR034")
-					(unit 1)
-				)

Commit message: Add files via upload
Parts:
- removed D2: IO_STATUS, LED_SMD:LED_0603_1608Metric, symbol Device:LED
- removed D3: POWER STATUS, LED_SMD:LED_0603_1608Metric, symbol Device:LED
- added C54: 100n, Capacitor_SMD:C_0603_1608Metric, symbol Device:C
- added R15: 4.7k, Resistor_SMD:R_0603_1608Metric, symbol Device:R
- added R16: 10k, Resistor_SMD:R_0603_1608Metric, symbol Device:R
- added R17: 10K, Resistor_SMD:R_0603_1608Metric, symbol Device:R
- added R18: 47K, Resistor_SMD:R_0603_1608Metric, symbol Device:R
- R11: value NC -> 22k; now fitted
- R6: value 33 -> 1k
- R7: value 100 -> 2.2k
Connections:
- net AIN0: now also U2.AL29 (AIN5/P0.26); no longer U2.V2 (AIN0/P0.04)
- net BCK: now also U2.AL9 (IO3/P0.16); no longer U2.B18 (P1.12)
- net DIN: now also U2.AL13 (P0.19); no longer U2.B16 (P1.14)
- net EC11_A: now also U2.A17 (P1.13); no longer U2.AK28 (AIN4/P0.25)
- net EC11_B: now also U2.AL19 (P1.04); no longer U2.AK26 (P1.09)
- net GND: now also C54.2; no longer SW2.2, SW3.2, SW4.2, SW5.2, SW6.S2, SW7.2
- net LRCK: now also U2.AL15 (P0.21); no longer U2.B14 (P1.15)
- net MISO: now also U2.AL5 (IO0/P0.13); no longer U2.AK2 (MISO/TRACEDATA1/P0.10)
- net SCK: now also U2.W1 (NFC1/P0.02); no longer U2.AH2 (SCK/TRACEDATA3/P0.08)
- net VDD: now also R11.1, R6.1, R7.1, R15.1, R16.1, R17.1, R18.1
- net VDDA: now also U6.13 (EN), U6.6 (G0), U6.7 (G1), U8.17 (XSMT)
- net at R6.2: now also SW2.1
- net at R7.2: now also SW3.1
- net BUTTONS: now reaches U2.AE31 (AIN7/P0.28)
- net BUTTONS: now also SW2.2, SW3.2, SW4.2, SW5.2, SW6.S2, SW7.2
- net EXIT: no longer names the net of SW4.1
- net EXIT: now also R15.2; no longer U2.AK20 (P0.23)
- net G0: no longer names the net of U2.B24 (P0.30)
- net G0: no longer U6.6 (G0)
- removed net G1: U2.A17 (P1.13), U6.7 (G1)
- net IO1: no longer names the net of U2.M2 (P1.00)
- net IO1: no longer R6.1
- net IO2: no longer names the net of U2.P2 (P1.01)
- net IO2: no longer R7.1
- net MUTE: no longer names the net of U2.B20 (P1.11)
- net MUTE: no longer U8.17 (XSMT)
- net OPTIONS: no longer names the net of U2.AK22 (P1.05)
- net OPTIONS: no longer SW5.1
- net PLAY/STOP: no longer names the net of U2.AK16 (P0.20)
- net PLAY/STOP: no longer SW2.1
- net POWER: no longer names the net of U2.AK6 (DCX/TRACECLK/P0.12)
- net POWER: no longer R11.1
- net RES: no longer names the net of U4.5 (RES)
- net RES: now also C54.1, R17.2; no longer U2.AL19 (P1.04)
- net SELECT: no longer names the net of U2.AK30 (AIN6/P0.27)
- net SELECT: no longer SW6.S1
- net SKIP: no longer names the net of U2.AK18 (P0.22)
- net SKIP: no longer SW3.1
- net TPA_EN: no longer names the net of U2.B22 (P0.31)
- net TPA_EN: no longer U6.13 (EN)
- new net: R16.2, SW5.1
- new net S1: R18.2, SW6.S1
- no-connect marks 20 -> 32
Other:
- note removed: "FINISH THE PCM5102A, TPA6132A2RTE, SJ43514, GND AND VDD SEPERATION, ANTENNA"
- moved on the sheet: SW2, SW3, SW4, SW5, SW7, U4
