File: Music-player.kicad_sch (KiCad schematic)
At the start: 102 parts, among them J1 USB_C_Receptacle_USB2.0_14P, J2 Screw_Terminal_01x04, J3 Screw_Terminal_01x02, J4 MSD-4-A, J5 SJ-43514, Q2 DMG2301L, SW1 RESET, SW2 PLAY/STOP, SW3 SKIP, SW4 EXIT, SW5 OPTIONS, SW6 EC11_L, SW7 POWER, U1 TVS1400DRV, U2 nRF5340-QKxx, U3 NCP1117-3.3_SOT223, U5 MCP73831-2-OT, U6 TPA6132A2RTE, U8 PCM5102A, Y1 MU00525-32-768K, Y2 ECS-320-8-37B-CKY-TR

Commit message: Add files via upload
Parts:
- removed R17: 10K, Resistor_SMD:R_0603_1608Metric, symbol Device:R
- removed U3: NCP1117-3.3_SOT223, Package_TO_SOT_SMD:SOT-223-3_TabPin2, symbol Regulator_Linear:NCP1117-3.3_SOT223
- added U3: SPX3819M5-L-3-3, Package_TO_SOT_SMD:SOT-23-5, symbol Regulator_Linear:SPX3819M5-L-3-3
- C54: value 100n -> 10n
- SW1: footprint MyFootprintLibrary:SW_K2-1107ST-A4DW-06_HRO -> myotherkicadfootprintlibrary:B3U-1000P
Connections:
- net CD: now also U2.W1 (NFC1/P0.02); no longer U2.AA1 (NFC2/P0.03)
- net GND: now also U3.2 (GND)
- net MISO: now also U2.AA1 (NFC2/P0.03); no longer U2.AL5 (IO0/P0.13)
- net MSD_CS: now also U2.AL5 (IO0/P0.13); no longer U2.AE1 (TWI/P1.02)
- net SCK: now also U2.AE1 (TWI/P1.02); no longer U2.W1 (NFC1/P0.02)
- net USB_POWER: now also U3.1 (IN), U3.3 (EN)
- net VDD: now also U3.5 (OUT)
- net at C54.1: now also U3.4 (BP); no longer U4.5 (RES)
- net RES: now reaches U2.U31 (P0.29)
- net RES: now also U4.5 (RES)
- no-connect marks 32 -> 2
Other:
- moved on the sheet: C2

Commit message: Add files via upload
Parts:
- added Q3: DMG2301L, Package_TO_SOT_SMD:SOT-23, symbol Transistor_FET:DMG2301L
Connections:
- net CHARGING: now also Q3.1 (G)
- net USB_POWER: now also Q3.3 (D); no longer C11.1, J3.2 (Pin_2), Q2.1 (G), U5.3 (V_{BAT})
- new net USB_GATE: C11.1, J3.2 (Pin_2), Q2.1 (G), Q3.2 (S), U5.3 (V_{BAT})
Other:
- note added: "C28 ST7789"
- note removed: "C28 SST7789"
Changed lines of the file:
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@@
 		)
 	)
-	(text "C28\nSST7789\n"
+	(text "C28\nST7789\n"
 		(exclude_from_sim no)
 		(at 260.35 115.57 0)
@@
 	)
 	(junction
+		(at 363.22 81.28)
+		(diameter 0)
+		(color 0 0 0 0)
+	)
+	(junction
 		(at 335.28 91.44)
 		(diameter 0)
@@
 	(wire
 		(pts
+			(xy 363.22 81.28) (xy 363.22 76.2)
+		)
+		(stroke
+			(width 0)
+			(type default)
+		)
+	)
+	(wire
+		(pts
 			(xy 383.54 45.72) (xy 383.54 66.04)
 		)
@@
 	(wire
 		(pts
+			(xy 368.3 73.66) (xy 368.3 72.39)
+		)
+		(stroke
+			(width 0)
+			(type default)
+		)
+	)
+	(wire
+		(pts
 			(xy 254 43.18) (xy 264.16 43.18)
 		)
@@
 	(wire
 		(pts
-			(xy 356.87 81.28) (xy 381 81.28)
+			(xy 356.87 81.28) (xy 363.22 81.28)
 		)
 		(stroke
@@
 	(wire
 		(pts
+			(xy 373.38 81.28) (xy 381 81.28)
+		)
+		(stroke
+			(width 0)
+			(type default)
+		)
+	)
+	(wire
+		(pts
 			(xy 304.8 113.03) (xy 311.15 113.03)
 		)
@@
 	(wire
 		(pts
-			(xy 384.81 20.32) (xy 389.89 20.32)
+			(xy 379.73 20.32) (xy 389.89 20.32)
 		)
 		(stroke
@@
 	(wire
 		(pts
+			(xy 363.22 76.2) (xy 355.6 76.2)
+		)
+		(stroke
+			(width 0)
+			(type default)
+		)
+	)
+	(wire
+		(pts
 			(xy 254 43.18) (xy 254 48.26)
 		)
@@
 	(wire
 		(pts
+			(xy 368.3 72.39) (xy 358.14 72.39)
+		)
+		(stroke
+			(width 0)
+			(type default)
+		)
+	)
+	(wire
+		(pts
 			(xy 163.83 128.27) (xy 152.4 128.27)
 		)
@@
 		)
 	)
+	(label "USB_GATE"
+		(at 355.6 76.2 0)
+		(effects
+			(font
+				(size 1.27 1.27)
+			)
+			(justify left bottom)
+		)
+	)
 	(label "EC11_A"
 		(at 185.42 80.01 0)
@@
 		)
 	)
+	(label "CHARGING"
+		(at 358.14 72.39 0)
+		(effects
+			(font
+				(size 1.27 1.27)
+			)
+			(justify left bottom)
+		)
+	)
 	(label "SWDIO"
 		(at 77.47 77.47 0)
@@
 		)
 	)
-	(label "VBAT"
+	(label "USB_GATE"
 		(at 398.78 102.87 180)
 		(effects
@@
 		)
 	)
-	(label "VBAT"
-		(at 384.81 20.32 0)
+	(label "USB_GATE"
+		(at 379.73 20.32 0)
 		(effects
 			(font
@@
 					(unit 1)
 				)
+			)
+		)
+	)
+	(symbol
+		(lib_id "Transistor_FET:DMG2301L")
+		(at 368.3 78.74 270)
+		(unit 1)
+		(body_style 1)
+		(exclude_from_sim no)
+		(in_bom yes)
+		(on_board yes)
+		(in_pos_files yes)
+		(dnp no)
+		(fields_autoplaced yes)
+		(property "Reference" "Q3"
+			(at 368.3 85.09 90)
+			(show_name no)
+			(do_not_autoplace no)
+			(effects
+				(font
+					(size 1.27 1.27)
+				)
+			)
+		)
+		(property "Value" "DMG2301L"
+			(at 368.3 87.63 90)
+			(show_name no)
+			(do_not_autoplace no)
+			(effects
+				(font
+					(size 1.27 1.27)
+				)
+			)
+		)
+		(property "Footprint" "Package_TO_SOT_SMD:SOT-23"
+			(at 366.395 83.82 0)
+			(hide yes)
+			(show_name no)
+			(do_not_autoplace no)
+			(effects
+				(font
+					(size 1.27 1.27)
+					(italic yes)
+				)
+				(justify left)
+			)
+		)
+		(property "Datasheet" "https://www.diodes.com/assets/Datasheets/DMG2301L.pdf"
+			(at 364.49 83.82 0)
+			(hide yes)
+			(show_name no)
+			(do_not_autoplace no)
+			(effects
+				(font
+					(size 1.27 1.27)
+				)
+				(justify left)
+			)
+		)
+		(property "Description" "-3A Id, -20V Vds, P-Channel MOSFET, SOT-23"
+			(at 368.3 78.74 0)
+			(hide yes)
+			(show_name no)
+			(do_not_autoplace no)
+			(effects
+				(font
+					(size 1.27 1.27)
+				)
+			)
+		)
+		(pin "1"
+		)
+		(pin "3"
+		)
+		(pin "2"
+		)
+		(instances
+			(project "Music-player"
+				(path "/f98d3056-e9c6-4dc5-a080-338d8b2650d2"
+					(reference "Q3")
+					(unit 1)
+				)

Commit message: Add files via upload
Connections:
- net BUTTONS: now also SW6.B; no longer SW6.S2
- net EC11_A: now also SW6.S1; no longer SW6.A
- net EC11_B: now also SW6.S2; no longer SW6.B
- net GND: no longer SW6.C
- net PCM_OUTL: now also C43.1; no longer C44.1
- net PCM_OUTR: now also C44.1; no longer C43.1
- net S1: now also SW6.A; no longer SW6.S1
Other:
- note added: "NET INTENTIONALLY SWAPPED COMPENSATE IN SOFTWARE"
Changed lines of the file:
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@@
 		)
 	)
+	(text "NET INTENTIONALLY SWAPPED\nCOMPENSATE IN SOFTWARE"
+		(exclude_from_sim no)
+		(at 199.898 218.44 0)
+		(effects
+			(font
+				(size 0.635 0.635)
+			)
+		)
+	)
 	(text "C27\nE1\n"
 		(exclude_from_sim no)
@@
 	(wire
 		(pts
-			(xy 378.46 232.41) (xy 378.46 231.14)
-		)
-		(stroke
-			(width 0)
-			(type default)
-		)
-	)
-	(wire
-		(pts
 			(xy 384.81 158.75) (xy 392.43 158.75)
 		)
@@
 	)
 	(label "PCM_OUTR"
-		(at 177.8 214.63 0)
+		(at 177.8 205.74 0)
 		(effects
 			(font
@@
 	)
 	(label "PCM_OUTL"
-		(at 177.8 205.74 0)
+		(at 177.8 214.63 0)
 		(effects
 			(font
@@
 		(lib_id "Device:RotaryEncoder_Switch")
 		(at 200.66 82.55 0)
+		(mirror y)
 		(unit 1)
 		(body_style 1)
@@
 		(in_pos_files yes)
 		(dnp no)
-		(fields_autoplaced yes)
 		(property "Reference" "SW6"
 			(at 200.66 72.39 0)
@@
 		)
 		(property "Footprint" "Rotary_Encoder:RotaryEncoder_Alps_EC11E-Switch_Vertical_H20mm_MountingHoles"
-			(at 196.85 78.486 0)
+			(at 204.47 78.486 0)
 			(hide yes)
 			(show_name no)
@@
 	(symbol
 		(lib_id "power:GND")
-		(at 378.46 231.14 0)
+		(at 378.46 232.41 0)
 		(unit 1)
 		(body_style 1)
@@
 		(fields_autoplaced yes)
 		(property "Reference" "#PWR026"
-			(at 378.46 237.49 0)
+			(at 378.46 238.76 0)
 			(hide yes)
 			(show_name no)
@@
 		)
 		(property "Value" "GND"
-			(at 378.46 236.22 0)
+			(at 378.46 237.49 0)
 			(hide yes)
 			(show_name no)
@@
 		)
 		(property "Footprint" ""
-			(at 378.46 231.14 0)
+			(at 378.46 232.41 0)
 			(hide yes)
 			(show_name no)
@@
 		)
 		(property "Datasheet" ""
-			(at 378.46 231.14 0)
+			(at 378.46 232.41 0)
 			(hide yes)
 			(show_name no)
@@
 		)
 		(property "Description" "Power symbol creates a global label with name \"GND\" , ground"
-			(at 378.46 231.14 0)
+			(at 378.46 232.41 0)
 			(hide yes)
 			(show_name no)

Commit message: Add files via upload
Parts:
- C23, C25, C4, C5: now not fitted
- Y1: value MU00525-32-768K -> Seiko SC-20S; footprint Crystal:Crystal_SMD_3215-2Pin_3.2x1.5mm -> Crystal:Crystal_SMD_2012-2Pin_2.0x1.2mm
- Y2: value ECS-320-8-37B-CKY-TR -> TXC 8Q32000002; footprint Crystal:Crystal_SMD_3225-4Pin_3.2x2.5mm -> MyFootprintLibrary:XTAL_8Q-32.000MEEV-T
Connections:
- net at C9.1, R4.2, U2.A5 (VBUS): now also C5.1, U2.B6 (DECUSB)
- net at C3.1, U2.A23 (DECN): now also C4.1, U2.A13 (DECA)
Other:
- note added: "ST7789 SCREEN"
- note removed: "SST7789 SCREEN"
Changed lines of the file:
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@@
 		)
 	)
-	(text "SST7789 SCREEN\n"
+	(text "ST7789 SCREEN\n"
 		(exclude_from_sim no)
 		(at 369.57 178.308 0)
@@
 	)
 	(junction
+		(at 67.31 201.93)
+		(diameter 0)
+		(color 0 0 0 0)
+	)
+	(junction
 		(at 181.61 265.43)
 		(diameter 0)
@@
 	)
 	(junction
+		(at 80.01 207.01)
+		(diameter 0)
+		(color 0 0 0 0)
+	)
+	(junction
 		(at 254 38.1)
 		(diameter 0)
@@
 	)
 	(junction
+		(at 86.36 207.01)
+		(diameter 0)
+		(color 0 0 0 0)
+	)
+	(junction
 		(at 209.55 105.41)
 		(diameter 0)
@@
 	)
 	(junction
+		(at 73.66 201.93)
+		(diameter 0)
+		(color 0 0 0 0)
+	)
+	(junction
 		(at 222.25 187.96)
 		(diameter 0)
@@
 	(wire
 		(pts
+			(xy 67.31 201.93) (xy 73.66 201.93)
+		)
+		(stroke
+			(width 0)
+			(type default)
+		)
+	)
+	(wire
+		(pts
 			(xy 302.26 83.82) (xy 302.26 86.36)
 		)
@@
 	(wire
 		(pts
+			(xy 80.01 207.01) (xy 86.36 207.01)
+		)
+		(stroke
+			(width 0)
+			(type default)
+		)
+	)
+	(wire
+		(pts
 			(xy 251.46 265.43) (xy 251.46 266.7)
 		)
@@
 	(wire
 		(pts
+			(xy 67.31 201.93) (xy 67.31 204.47)
+		)
+		(stroke
+			(width 0)
+			(type default)
+		)
+	)
+	(wire
+		(pts
 			(xy 302.26 91.44) (xy 312.42 91.44)
 		)
@@
 	(wire
 		(pts
-			(xy 67.31 199.39) (xy 67.31 204.47)
+			(xy 67.31 199.39) (xy 67.31 201.93)
 		)
 		(stroke
@@
 		(on_board yes)
 		(in_pos_files yes)
-		(dnp no)
+		(dnp yes)
 		(property "Reference" "C23"
 			(at 228.6 107.442 0)
@@
 		(on_board yes)
 		(in_pos_files yes)
-		(dnp no)
+		(dnp yes)
 		(property "Reference" "C25"
 			(at 241.3 107.442 0)
@@
 		(on_board yes)
 		(in_pos_files yes)
-		(dnp no)
+		(dnp yes)
 		(property "Reference" "C5"
 			(at 73.914 207.772 0)
@@
 		(on_board yes)
 		(in_pos_files yes)
-		(dnp no)
+		(dnp yes)
 		(property "Reference" "C4"
 			(at 86.614 210.058 0)
@@
 			)
 		)
-		(property "Value" "MU00525-32-768K"
+		(property "Value" "Seiko SC-20S"
 			(at 149.86 35.5599 90)
 			(show_name no)
@@
 			)
 		)
-		(property "Footprint" "Crystal:Crystal_SMD_3215-2Pin_3.2x1.5mm"
+		(property "Footprint" "Crystal:Crystal_SMD_2012-2Pin_2.0x1.2mm"
 			(at 147.32 34.29 0)
 			(hide yes)
@@
 			)
 		)
-		(property "Value" "ECS-320-8-37B-CKY-TR"
+		(property "Value" "TXC 8Q32000002"
 			(at 145.542 22.606 90)
 			(show_name no)
@@
 			)
 		)
-		(property "Footprint" "Crystal:Crystal_SMD_3225-4Pin_3.2x2.5mm"
+		(property "Footprint" "MyFootprintLibrary:XTAL_8Q-32.000MEEV-T"
 			(at 147.32 26.67 0)
 			(hide yes)

Commit message: Add files via upload
Parts:
- removed J1: USB_C_Receptacle_USB2.0_14P, Connector_USB:USB_C_Receptacle_GCT_USB4105-xx-A_16P_TopMnt_Horizontal, symbol Connector:USB_C_Receptacle_USB2.0_14P
- removed U1: TVS1400DRV, Package_SON:WSON-6-1EP_2x2mm_P0.65mm_EP1x1.6mm, symbol Power_Protection:TVS1400DRV
- added D2: PRTR5V0U2X, Package_TO_SOT_SMD:SOT-143, symbol Power_Protection:PRTR5V0U2X
- added J1: USB_C_Receptacle_USB2.0_16P, Connector_USB:USB_C_Receptacle_GCT_USB4105-xx-A_16P_TopMnt_Horizontal, symbol Connector:USB_C_Receptacle_USB2.0_16P
- E1: value 2450AT18B100E -> 2450AT43B100E; footprint MyFootprintLibrary:XDCR_2450AT18B100E -> MyFootprintLibrary:ANTENNA_2450AT43B100E
- FB1: value BLM18PG221SN1D -> TDK MPZ1608S221ATA00
Connections:
- net D+: now also D2.3 (I/O2), J1.A6 (D+), J1.B6 (D+)
- net D-: now also D2.2 (I/O1), J1.A7 (D-), J1.B7 (D-)
- net GND: now also D2.1 (GND), J1.A1 (GND), J1.A12 (GND), J1.A8 (SBU1), J1.B1 (GND), J1.B12 (GND), J1.B8 (SBU2), J1.SH (SHIELD)
- net at R2.1: now also J1.A5 (CC1)
- net at R1.1: now also J1.B5 (CC2)
- net CHARGING renamed VBUS
- net VBUS: now also D2.4 (VCC), J1.A4 (VBUS), J1.A9 (VBUS), J1.B4 (VBUS), J1.B9 (VBUS)

Commit message: Add files via upload
Parts:
- C10, C12, C13, C14, C16, C17, C18, C19, C20, C21, C22, C23, C24, C25, C28, C29, C3, C30, C31, C32, C33, C34, C35, C36, C38, C39, C4, C40, C41, C42, C43, C44, C45, C46, C47, C48, C50, C51, C52, C53, C54, C7, C8: footprint Capacitor_SMD:C_0603_1608Metric -> Capacitor_SMD:C_0402_1005Metric
- L1, L2, L3: footprint Inductor_SMD:L_0201_0603Metric -> Inductor_SMD:L_0603_1608Metric
- R1, R10, R11, R12, R13, R14, R15, R16, R18, R2, R3, R4, R5, R6, R7, R8, R9: footprint Resistor_SMD:R_0603_1608Metric -> Resistor_SMD:R_0402_1005Metric

Commit message: Add files via upload
Parts:
- removed Y2: TXC 8Q32000002, MyFootprintLibrary:XTAL_8Q-32.000MEEV-T, symbol Device:Crystal_Small
- added Y2: TXC 8Q32000002, myotherkicadfootprintlibrary:XTAL_8Q-32.000MEEV-T, symbol Device:Crystal_GND24
Connections:
- net DC: now also U2.A17 (P1.13); no longer U2.AL21 (P1.06)
- net EC11_A: now also U2.U31 (P0.29); no longer U2.A17 (P1.13)
- net GND: now also Y2.2 (G), Y2.4 (G)
- net RES: now also U2.AL21 (P1.06); no longer U2.U31 (P0.29)
- net XC1: now also Y2.3
- net XC2: now also Y2.1
Other:
- moved on the sheet: Y1
Changed lines of the file:
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@@
 	(wire
 		(pts
+			(xy 147.32 21.59) (xy 147.32 22.86)
+		)
+		(stroke
+			(width 0)
+			(type default)
+		)
+	)
+	(wire
+		(pts
 			(xy 215.9 240.03) (xy 220.98 240.03)
 		)
@@
 	(wire
 		(pts
-			(xy 140.97 36.83) (xy 147.32 36.83)
+			(xy 140.97 40.64) (xy 147.32 40.64)
 		)
 		(stroke
@@
 	(wire
 		(pts
-			(xy 140.97 29.21) (xy 147.32 29.21)
+			(xy 140.97 31.75) (xy 147.32 31.75)
 		)
 		(stroke
@@
 	(wire
 		(pts
-			(xy 140.97 24.13) (xy 147.32 24.13)
+			(xy 140.97 21.59) (xy 147.32 21.59)
 		)
 		(stroke
@@
 	(wire
 		(pts
+			(xy 139.7 26.67) (xy 142.24 26.67)
+		)
+		(stroke
+			(width 0)
+			(type default)
+		)
+	)
+	(wire
+		(pts
 			(xy 290.83 76.2) (xy 294.64 76.2)
 		)
@@
 	(wire
 		(pts
+			(xy 147.32 31.75) (xy 147.32 30.48)
+		)
+		(stroke
+			(width 0)
+			(type default)
+		)
+	)
+	(wire
+		(pts
 			(xy 254 105.41) (xy 260.35 105.41)
 		)
@@
 	(wire
 		(pts
-			(xy 140.97 31.75) (xy 147.32 31.75)
+			(xy 140.97 35.56) (xy 147.32 35.56)
 		)
 		(stroke
@@
 	)
 	(label "XC2"
-		(at 140.97 29.21 0)
+		(at 140.97 21.59 0)
 		(effects
 			(font
@@
 	)
 	(label "DC"
-		(at 163.83 173.99 180)
+		(at 163.83 191.77 180)
 		(effects
 			(font
@@
 	)
 	(label "XL1"
-		(at 140.97 31.75 0)
+		(at 140.97 35.56 0)
 		(effects
 			(font
@@
 	)
 	(label "EC11_A"
-		(at 163.83 191.77 180)
+		(at 163.83 148.59 180)
 		(effects
 			(font
@@
 	)
 	(label "RES"
-		(at 163.83 148.59 180)
+		(at 163.83 173.99 180)
 		(effects
 			(font
@@
 	)
 	(label "XL2"
-		(at 140.97 36.83 0)
+		(at 140.97 40.64 0)
 		(effects
 			(font
@@
 	)
 	(label "XC1"
-		(at 140.97 24.13 0)
+		(at 140.97 31.75 0)
 		(effects
 			(font
@@
 	)
 	(symbol
+		(lib_id "power:GND")
+		(at 139.7 26.67 0)
+		(mirror y)
+		(unit 1)
+		(body_style 1)
+		(exclude_from_sim no)
+		(in_bom yes)
+		(on_board yes)
+		(in_pos_files yes)
+		(dnp no)
+		(property "Reference" "#PWR034"
+			(at 139.7 33.02 0)
+			(hide yes)
+			(show_name no)
+			(do_not_autoplace no)
+			(effects
+				(font
+					(size 1.27 1.27)
+				)
+			)
+		)
+		(property "Value" "GND"
+			(at 139.7 31.75 0)
+			(hide yes)
+			(show_name no)
+			(do_not_autoplace no)
+			(effects
+				(font
+					(size 1.27 1.27)
+				)
+			)
+		)
+		(property "Footprint" ""
+			(at 139.7 26.67 0)
+			(hide yes)
+			(show_name no)
+			(do_not_autoplace no)
+			(effects
+				(font
+					(size 1.27 1.27)
+				)
+			)
+		)
+		(property "Datasheet" ""
+			(at 139.7 26.67 0)
+			(hide yes)
+			(show_name no)
+			(do_not_autoplace no)
+			(effects
+				(font
+					(size 1.27 1.27)
+				)
+			)
+		)
+		(property "Description" "Power symbol creates a global label with name \"GND\" , ground"
+			(at 139.7 26.67 0)
+			(hide yes)
+			(show_name no)
+			(do_not_autoplace no)
+			(effects
+				(font
+					(size 1.27 1.27)
+				)
+			)
+		)
+		(pin "1"
+		)
+		(instances
+			(project "Music-player"
+				(path "/f98d3056-e9c6-4dc5-a080-338d8b2650d2"
+					(reference "#PWR034")
+					(unit 1)
+				)
+			)
+		)
+	)
+	(symbol
 		(lib_id "Device:C")
 		(at 86.36 212.09 0)
@@
 	(symbol
 		(lib_id "Device:Crystal_Small")
-		(at 147.32 34.29 90)
+		(at 147.32 38.1 90)
 		(unit 1)
 		(body_style 1)
@@
 		(fields_autoplaced yes)
 		(property "Reference" "Y1"
-			(at 149.86 33.0199 90)
+			(at 149.86 36.8299 90)
 			(show_name no)
 			(do_not_autoplace no)
@@
 		)
 		(property "Value" "Seiko SC-20S"
-			(at 149.86 35.5599 90)
+			(at 149.86 39.3699 90)
 			(show_name no)
 			(do_not_autoplace no)
@@
 		)
 		(property "Footprint" "Crystal:Crystal_SMD_2012-2Pin_2.0x1.2mm"
-			(at 147.32 34.29 0)
+			(at 147.32 38.1 0)
 			(hide yes)
 			(show_name no)
@@
 		)
 		(property "Datasheet" ""
-			(at 147.32 34.29 0)
+			(at 147.32 38.1 0)
 			(hide yes)
 			(show_name no)
@@
 		)
 		(property "Description" "Two pin crystal, small symbol"
-			(at 147.32 34.29 0)
+			(at 147.32 38.1 0)
 			(hide yes)
 			(show_name no)
@@
 	)
 	(symbol
-		(lib_id "Device:Crystal_Small")
-		(at 147.32 26.67 270)
-		(unit 1)
-		(body_style 1)
-		(exclude_from_sim no)
-		(in_bom yes)
-		(on_board yes)
-		(in_pos_files yes)
-		(dnp no)
-		(property "Reference" "Y2"
-			(at 149.86 25.3999 90)
-			(show_name no)
-			(do_not_autoplace no)
-			(effects
-				(font
-					(size 1.27 1.27)
-				)
-				(justify left)
-			)
-		)
-		(property "Value" "TXC 8Q32000002"
-			(at 145.542 22.606 90)
-			(show_name no)
-			(do_not_autoplace no)
-			(effects
-				(font
-					(size 1.27 1.27)
-				)
-				(justify left)
-			)
-		)
-		(property "Footprint" "MyFootprintLibrary:XTAL_8Q-32.000MEEV-T"
-			(at 147.32 26.67 0)
-			(hide yes)
-			(show_name no)
-			(do_not_autoplace no)
-			(effects
-				(font
-					(size 1.27 1.27)
-				)
-			)
-		)
-		(property "Datasheet" ""
-			(at 147.32 26.67 0)
-			(hide yes)
-			(show_name no)
-			(do_not_autoplace no)
-			(effects
-				(font
-					(size 1.27 1.27)
-				)
-			)
-		)
-		(property "Description" "Two pin crystal, small symbol"
-			(at 147.32 26.67 0)
-			(hide yes)
-			(show_name no)
-			(do_not_autoplace no)
-			(effects
-				(font
-					(size 1.27 1.27)
-				)
-			)
-		)
-		(pin "2"
-		)
-		(pin "1"
-		)
-		(instances
-			(project "Music-player"
-				(path "/f98d3056-e9c6-4dc5-a080-338d8b2650d2"
-					(reference "Y2")
-					(unit 1)
-				)
-			)
-		)
-	)
-	(symbol
 		(lib_id "Device:C")
 		(at 247.65 246.38 0)
@@
 					(unit 1)
 				)
+			)
+		)
+	)
+	(symbol
+		(lib_id "Device:Crystal_GND24")
+		(at 147.32 26.67 270)
+		(unit 1)
+		(body_style 1)
+		(exclude_from_sim no)
+		(in_bom yes)
+		(on_board yes)
+		(in_pos_files yes)
+		(dnp no)
+		(fields_autoplaced yes)
+		(property "Reference" "Y2"
+			(at 152.4 25.3999 90)
+			(show_name no)
+			(do_not_autoplace no)
+			(effects
+				(font
+					(size 1.27 1.27)
+				)
+				(justify left)
+			)
+		)
+		(property "Value" "TXC 8Q32000002"
+			(at 152.4 27.9399 90)
+			(show_name no)
+			(do_not_autoplace no)
+			(effects
+				(font
+					(size 1.27 1.27)
+				)
+				(justify left)
+			)
+		)
+		(property "Footprint" "myotherkicadfootprintlibrary:XTAL_8Q-32.000MEEV-T"
+			(at 147.32 26.67 0)
+			(hide yes)
+			(show_name no)
+			(do_not_autoplace no)
+			(effects
+				(font
+					(size 1.27 1.27)
+				)
+			)
+		)
+		(property "Datasheet" ""
+			(at 147.32 26.67 0)
+			(hide yes)
+			(show_name no)
+			(do_not_autoplace no)
+			(effects
+				(font
+					(size 1.27 1.27)
+				)
+			)
+		)
+		(property "Description" "Four pin crystal, GND on pins 2 and 4"
+			(at 147.32 26.67 0)
+			(hide yes)
+			(show_name no)
+			(do_not_autoplace no)
+			(effects
+				(font
+					(size 1.27 1.27)
+				)
+			)
+		)
+		(property private "KLC_S3.3" "The rectangle is not a symbol body but a graphical element"
+			(at 134.62 26.67 0)
+			(hide yes)
+			(show_name yes)
+			(do_not_autoplace no)
+			(effects
+				(font
+					(size 1.27 1.27)
+				)
+			)
+		)
+		(property private "KLC_S4.1" "Some pins are on 50mil grid to make the symbol small"
+			(at 132.08 26.67 0)
+			(hide yes)
+			(show_name yes)
+			(do_not_autoplace no)
+			(effects
+				(font
+					(size 1.27 1.27)
+				)
+			)
+		)
+		(pin "2"
+		)
+		(pin "3"
+		)
+		(pin "1"
+		)
+		(pin "4"
+		)
+		(instances
+			(project "Music-player"
+				(path "/f98d3056-e9c6-4dc5-a080-338d8b2650d2"
+					(reference "Y2")
+					(unit 1)
+				)

Commit message: Add files via upload
Parts:
- C15: footprint Capacitor_SMD:C_0603_1608Metric -> Capacitor_SMD:C_0402_1005Metric
- L1, L2, L3: footprint Inductor_SMD:L_0603_1608Metric -> Inductor_SMD:L_0402_1005Metric
- Y2: value TXC 8Q32000002 -> NX2016SA-CS06654; footprint myotherkicadfootprintlibrary:XTAL_8Q-32.000MEEV-T -> MyFootprintLibrary:NX2016SA_NDK
Connections:
- net BLK: now also U2.A17 (P1.13); no longer U2.AL27 (P0.24)
- net DC: now also U2.AL23 (P1.08); no longer U2.A17 (P1.13)
- net RES: now also U2.AL27 (P0.24); no longer U2.AL21 (P1.06)
- net SST_CS: now also U2.AL21 (P1.06); no longer U2.AL23 (P1.08)
Changed lines of the file:
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@@
 	)
 	(label "DC"
-		(at 163.83 191.77 180)
+		(at 163.83 179.07 180)
 		(effects
 			(font
@@
 	)
 	(label "RES"
-		(at 163.83 173.99 180)
+		(at 163.83 135.89 180)
 		(effects
 			(font
@@
 	)
 	(label "BLK"
-		(at 163.83 135.89 180)
+		(at 163.83 191.77 180)
 		(effects
 			(font
@@
 	)
 	(label "SST_CS"
-		(at 163.83 179.07 180)
+		(at 163.83 173.99 180)
 		(effects
 			(font
@@
 			)
 		)
-		(property "Footprint" "Inductor_SMD:L_0603_1608Metric"
+		(property "Footprint" "Inductor_SMD:L_0402_1005Metric"
 			(at 123.19 64.77 0)
 			(hide yes)
@@
 			)
 		)
-		(property "Footprint" "Inductor_SMD:L_0603_1608Metric"
+		(property "Footprint" "Inductor_SMD:L_0402_1005Metric"
 			(at 72.39 130.81 0)
 			(hide yes)
@@
 			)
 		)
-		(property "Footprint" "Capacitor_SMD:C_0603_1608Metric"
+		(property "Footprint" "Capacitor_SMD:C_0402_1005Metric"
 			(at 74.6252 191.77 0)
 			(hide yes)
@@
 			)
 		)
-		(property "Value" "TXC 8Q32000002"
+		(property "Value" "NX2016SA-CS06654"
 			(at 152.4 27.9399 90)
 			(show_name no)
@@
 			)
 		)
-		(property "Footprint" "myotherkicadfootprintlibrary:XTAL_8Q-32.000MEEV-T"
+		(property "Footprint" "MyFootprintLibrary:NX2016SA_NDK"
 			(at 147.32 26.67 0)
 			(hide yes)
@@
 			)
 		)
-		(property "Footprint" "Inductor_SMD:L_0603_1608Metric"
+		(property "Footprint" "Inductor_SMD:L_0402_1005Metric"
 			(at 72.39 161.29 0)
 			(hide yes)
