File: Music-player.kicad_sch (KiCad schematic)
At the start: 102 parts, among them J1 USB_C_Receptacle_USB2.0_16P, J2 Screw_Terminal_01x04, J3 Screw_Terminal_01x02, J4 MSD-4-A, J5 SJ-43514, Q2 DMG2301L, Q3 DMG2301L, SW1 RESET, SW2 PLAY/STOP, SW3 SKIP, SW4 EXIT, SW5 OPTIONS, SW6 EC11_L, SW7 POWER, U2 nRF5340-QKxx, U3 SPX3819M5-L-3-3, U5 MCP73831-2-OT, U6 TPA6132A2RTE, U8 PCM5102A, Y1 Seiko SC-20S, Y2 NX2016SA-CS06654

Commit message: Add files via upload
Parts:
- removed R18: 47K, Resistor_SMD:R_0402_1005Metric, symbol Device:R
- removed SW2: PLAY/STOP, MyFootprintLibrary:SW_K2-1107ST-A4DW-06_HRO, symbol Switch:SW_Push
- removed SW3: SKIP, MyFootprintLibrary:SW_K2-1107ST-A4DW-06_HRO, symbol Switch:SW_Push
- removed SW4: EXIT, MyFootprintLibrary:SW_K2-1107ST-A4DW-06_HRO, symbol Switch:SW_Push
- removed SW5: OPTIONS, MyFootprintLibrary:SW_K2-1107ST-A4DW-06_HRO, symbol Switch:SW_Push
- removed SW6: EC11_L, Rotary_Encoder:RotaryEncoder_Alps_EC11E-Switch_Vertical_H20mm_MountingHoles, symbol Device:RotaryEncoder_Switch
- removed SW7: POWER, MyFootprintLibrary:SW_K2-1107ST-A4DW-06_HRO, symbol Switch:SW_Push
- added U1: (no value), Connector_PinHeader_2.54mm:PinHeader_1x09_P2.54mm_Vertical, symbol New_Library:pinheader
Connections:
- net BUTTONS is gone; now on net BTN: U2.AE31 (AIN7/P0.28)
- net VDD: now also U1.3 (COMA), U1.9 (COMB); no longer R11.1, R15.1, R16.1, R6.1, R7.1
- net BTN: now reaches R15.2
- net BTN: now also R11.2, R16.2, R6.2, R7.2
- net EC11_A renamed ENCB
- net ENCB: now also U1.2 (ENCB)
- net EC11_B renamed ENCA
- net ENCA: now also U1.1 (ENCA)
- new net: R15.1, U1.6 (SW3)
- new net: R11.1, U1.8 (SW5)
- new net: R6.1, U1.4 (SW1)
- new net: R7.1, U1.5 (SW2)
- new net: R16.1, U1.7 (SW4)
Other:
- moved on the sheet: R11, R15, R16, R6, R7

Commit message: Add files via upload
Parts:
- C23, C4: now fitted
Connections:
- net at C3.1, U2.A23 (DECN): no longer C4.1, U2.A13 (DECA)
- new net: C4.1, U2.A13 (DECA)
Changed lines of the file:
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@@
 	)
 	(junction
-		(at 80.01 207.01)
-		(diameter 0)
-		(color 0 0 0 0)
-	)
-	(junction
 		(at 72.39 156.21)
 		(diameter 0)
@@
 	)
 	(junction
-		(at 86.36 207.01)
-		(diameter 0)
-		(color 0 0 0 0)
-	)
-	(junction
 		(at 209.55 105.41)
 		(diameter 0)
@@
 	(wire
 		(pts
-			(xy 80.01 207.01) (xy 86.36 207.01)
-		)
-		(stroke
-			(width 0)
-			(type default)
-		)
-	)
-	(wire
-		(pts
 			(xy 251.46 265.43) (xy 251.46 266.7)
 		)
@@
 		(on_board yes)
 		(in_pos_files yes)
-		(dnp yes)
+		(dnp no)
 		(property "Reference" "C23"
 			(at 228.6 107.442 0)
@@
 		(on_board yes)
 		(in_pos_files yes)
-		(dnp yes)
+		(dnp no)
 		(property "Reference" "C4"
 			(at 86.614 210.058 0)

Commit message: Add files via upload
Parts:
- added C55: 100n, Capacitor_SMD:C_0402_1005Metric, symbol Device:C
- J2: value Screw_Terminal_01x04 -> CONTACTS; footprint TerminalBlock_Phoenix:TerminalBlock_Phoenix_PT-1,5-4-3.5-H_1x04_P3.50mm_Horizontal -> Connector_PinHeader_2.54mm:PinHeader_1x04_P2.54mm_Vertical
Connections:
- net GND: now also C55.2
- net VDD: now also C55.1
Other:
- note added: "C16-C23 C55 VDD"
- note added: "PULL UP ON RESET"
- note removed: "C16-C23 VDD"
Changed lines of the file:
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@@
 	)
 	(rectangle
-		(start 177.8 97.79)
+		(start 173.99 97.79)
 		(end 340.36 120.65)
 		(stroke
@@
 		)
 	)
+	(text "PULL UP ON RESET\n"
+		(exclude_from_sim no)
+		(at 389.89 170.688 0)
+		(effects
+			(font
+				(size 1.27 1.27)
+			)
+		)
+	)
 	(text "CRYSTALS\n\n"
 		(exclude_from_sim no)
@@
 		)
 	)
-	(text "C16-C23\nVDD\n"
+	(text "C16-C23 C55\nVDD\n"
 		(exclude_from_sim no)
 		(at 208.28 115.57 0)
@@
 	)
 	(junction
+		(at 184.15 113.03)
+		(diameter 0)
+		(color 0 0 0 0)
+	)
+	(junction
 		(at 172.72 265.43)
 		(diameter 0)
@@
 	)
 	(junction
+		(at 184.15 105.41)
+		(diameter 0)
+		(color 0 0 0 0)
+	)
+	(junction
 		(at 317.5 76.2)
 		(diameter 0)
@@
 	(wire
 		(pts
+			(xy 177.8 113.03) (xy 184.15 113.03)
+		)
+		(stroke
+			(width 0)
+			(type default)
+		)
+	)
+	(wire
+		(pts
 			(xy 372.11 55.88) (xy 378.46 55.88)
 		)
@@
 	(wire
 		(pts
+			(xy 177.8 105.41) (xy 184.15 105.41)
+		)
+		(stroke
+			(width 0)
+			(type default)
+		)
+	)
+	(wire
+		(pts
 			(xy 368.3 72.39) (xy 358.14 72.39)
 		)
@@
 	)
 	(symbol
+		(lib_id "Device:C")
+		(at 177.8 109.22 0)
+		(unit 1)
+		(body_style 1)
+		(exclude_from_sim no)
+		(in_bom yes)
+		(on_board yes)
+		(in_pos_files yes)
+		(dnp no)
+		(property "Reference" "C55"
+			(at 177.8 107.442 0)
+			(show_name no)
+			(do_not_autoplace no)
+			(effects
+				(font
+					(size 1.27 1.27)
+				)
+				(justify left)
+			)
+		)
+		(property "Value" "100n"
+			(at 177.8 111.252 0)
+			(show_name no)
+			(do_not_autoplace no)
+			(effects
+				(font
+					(size 1.27 1.27)
+				)
+				(justify left)
+			)
+		)
+		(property "Footprint" "Capacitor_SMD:C_0402_1005Metric"
+			(at 178.7652 113.03 0)
+			(hide yes)
+			(show_name no)
+			(do_not_autoplace no)
+			(effects
+				(font
+					(size 1.27 1.27)
+				)
+			)
+		)
+		(property "Datasheet" ""
+			(at 177.8 109.22 0)
+			(hide yes)
+			(show_name no)
+			(do_not_autoplace no)
+			(effects
+				(font
+					(size 1.27 1.27)
+				)
+			)
+		)
+		(property "Description" "Unpolarized capacitor"
+			(at 177.8 109.22 0)
+			(hide yes)
+			(show_name no)
+			(do_not_autoplace no)
+			(effects
+				(font
+					(size 1.27 1.27)
+				)
+			)
+		)
+		(pin "1"
+		)
+		(pin "2"
+		)
+		(instances
+			(project "Music-player"
+				(path "/f98d3056-e9c6-4dc5-a080-338d8b2650d2"
+					(reference "C55")
+					(unit 1)
+				)
+			)
+		)
+	)
+	(symbol
 		(lib_id "Device:R")
 		(at 387.35 118.11 0)
@@
 			)
 		)
-		(property "Value" "Screw_Terminal_01x04"
+		(property "Value" "CONTACTS"
 			(at 232.41 74.93 0)
 			(show_name no)
@@
 			)
 		)
-		(property "Footprint" "TerminalBlock_Phoenix:TerminalBlock_Phoenix_PT-1,5-4-3.5-H_1x04_P3.50mm_Horizontal"
+		(property "Footprint" "Connector_PinHeader_2.54mm:PinHeader_1x04_P2.54mm_Vertical"
 			(at 232.41 83.82 0)
 			(hide yes)

Commit message: Add files via upload
Parts:
- added C56, C57, C58, C59: 100n, Capacitor_SMD:C_0402_1005Metric, symbol Device:C
- Y2: footprint MyFootprintLibrary:NX2016SA_NDK -> myotherkicadfootprintlibrary:NX2016SA_NDK
Connections:
- net GND: now also C56.2, C57.2, C58.2, C59.2
- net VDD: now also C56.1, C57.1, C58.1, C59.1

Commit message: Add files via upload
Parts:
- removed J2: CONTACTS, Connector_PinHeader_2.54mm:PinHeader_1x04_P2.54mm_Vertical, symbol Connector:Screw_Terminal_01x04
- added J2: Screw_Terminal_01x03, Connector_PinHeader_2.54mm:PinHeader_1x03_P2.54mm_Vertical, symbol Connector:Screw_Terminal_01x03
Connections:
- net GND: now also J2.1 (Pin_1)
- net SWDCLK: now also J2.3 (Pin_3)
- net SWDIO: now also J2.2 (Pin_2)
Changed lines of the file:
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@@
 	(wire
 		(pts
-			(xy 237.49 86.36) (xy 248.92 86.36)
-		)
-		(stroke
-			(width 0)
-			(type default)
-		)
-	)
-	(wire
-		(pts
 			(xy 196.85 113.03) (xy 203.2 113.03)
 		)
@@
 	(wire
 		(pts
-			(xy 237.49 83.82) (xy 248.92 83.82)
+			(xy 237.49 83.82) (xy 246.38 83.82)
 		)
 		(stroke
@@
 	)
 	(label "SWDIO"
-		(at 246.38 78.74 180)
+		(at 246.38 81.28 180)
 		(effects
 			(font
@@
 	)
 	(label "SWDCLK"
-		(at 246.38 81.28 180)
+		(at 246.38 78.74 180)
 		(effects
 			(font
@@
 	)
 	(symbol
-		(lib_id "power:GND")
-		(at 248.92 86.36 0)
-		(unit 1)
-		(body_style 1)
-		(exclude_from_sim no)
-		(in_bom yes)
-		(on_board yes)
-		(in_pos_files yes)
-		(dnp no)
-		(fields_autoplaced yes)
-		(property "Reference" "#PWR09"
-			(at 248.92 92.71 0)
-			(hide yes)
-			(show_name no)
-			(do_not_autoplace no)
-			(effects
-				(font
-					(size 1.27 1.27)
-				)
-			)
-		)
-		(property "Value" "GND"
-			(at 248.92 91.44 0)
-			(hide yes)
-			(show_name no)
-			(do_not_autoplace no)
-			(effects
-				(font
-					(size 1.27 1.27)
-				)
-			)
-		)
-		(property "Footprint" ""
-			(at 248.92 86.36 0)
-			(hide yes)
-			(show_name no)
-			(do_not_autoplace no)
-			(effects
-				(font
-					(size 1.27 1.27)
-				)
-			)
-		)
-		(property "Datasheet" ""
-			(at 248.92 86.36 0)
-			(hide yes)
-			(show_name no)
-			(do_not_autoplace no)
-			(effects
-				(font
-					(size 1.27 1.27)
-				)
-			)
-		)
-		(property "Description" "Power symbol creates a global label with name \"GND\" , ground"
-			(at 248.92 86.36 0)
-			(hide yes)
-			(show_name no)
-			(do_not_autoplace no)
-			(effects
-				(font
-					(size 1.27 1.27)
-				)
-			)
-		)
-		(pin "1"
-		)
-		(instances
-			(project "Music-player"
-				(path "/f98d3056-e9c6-4dc5-a080-338d8b2650d2"
-					(reference "#PWR09")
-					(unit 1)
-				)
-			)
-		)
-	)
-	(symbol
 		(lib_id "power:VDD")
 		(at 228.6 203.2 0)
@@
 	)
 	(symbol
+		(lib_id "power:GND")
+		(at 246.38 83.82 0)
+		(unit 1)
+		(body_style 1)
+		(exclude_from_sim no)
+		(in_bom yes)
+		(on_board yes)
+		(in_pos_files yes)
+		(dnp no)
+		(fields_autoplaced yes)
+		(property "Reference" "#PWR09"
+			(at 246.38 90.17 0)
+			(hide yes)
+			(show_name no)
+			(do_not_autoplace no)
+			(effects
+				(font
+					(size 1.27 1.27)
+				)
+			)
+		)
+		(property "Value" "GND"
+			(at 246.38 88.9 0)
+			(show_name no)
+			(do_not_autoplace no)
+			(effects
+				(font
+					(size 1.27 1.27)
+				)
+			)
+		)
+		(property "Footprint" ""
+			(at 246.38 83.82 0)
+			(hide yes)
+			(show_name no)
+			(do_not_autoplace no)
+			(effects
+				(font
+					(size 1.27 1.27)
+				)
+			)
+		)
+		(property "Datasheet" ""
+			(at 246.38 83.82 0)
+			(hide yes)
+			(show_name no)
+			(do_not_autoplace no)
+			(effects
+				(font
+					(size 1.27 1.27)
+				)
+			)
+		)
+		(property "Description" "Power symbol creates a global label with name \"GND\" , ground"
+			(at 246.38 83.82 0)
+			(hide yes)
+			(show_name no)
+			(do_not_autoplace no)
+			(effects
+				(font
+					(size 1.27 1.27)
+				)
+			)
+		)
+		(pin "1"
+		)
+		(instances
+			(project "Music-player"
+				(path "/f98d3056-e9c6-4dc5-a080-338d8b2650d2"
+					(reference "#PWR09")
+					(unit 1)
+				)
+			)
+		)
+	)
+	(symbol
 		(lib_id "power:GNDA")
 		(at 151.13 265.43 0)
@@
 	)
 	(symbol
-		(lib_id "power:VDD")
-		(at 248.92 83.82 0)
-		(unit 1)
-		(body_style 1)
-		(exclude_from_sim no)
-		(in_bom yes)
-		(on_board yes)
-		(in_pos_files yes)
-		(dnp no)
-		(fields_autoplaced yes)
-		(property "Reference" "#PWR032"
-			(at 248.92 87.63 0)
-			(hide yes)
-			(show_name no)
-			(do_not_autoplace no)
-			(effects
-				(font
-					(size 1.27 1.27)
-				)
-			)
-		)
-		(property "Value" "VDD"
-			(at 248.92 78.74 0)
-			(show_name no)
-			(do_not_autoplace no)
-			(effects
-				(font
-					(size 1.27 1.27)
-				)
-			)
-		)
-		(property "Footprint" ""
-			(at 248.92 83.82 0)
-			(hide yes)
-			(show_name no)
-			(do_not_autoplace no)
-			(effects
-				(font
-					(size 1.27 1.27)
-				)
-			)
-		)
-		(property "Datasheet" ""
-			(at 248.92 83.82 0)
-			(hide yes)
-			(show_name no)
-			(do_not_autoplace no)
-			(effects
-				(font
-					(size 1.27 1.27)
-				)
-			)
-		)
-		(property "Description" "Power symbol creates a global label with name \"VDD\""
-			(at 248.92 83.82 0)
-			(hide yes)
-			(show_name no)
-			(do_not_autoplace no)
-			(effects
-				(font
-					(size 1.27 1.27)
-				)
-			)
-		)
-		(pin "1"
-		)
-		(instances
-			(project "Music-player"
-				(path "/f98d3056-e9c6-4dc5-a080-338d8b2650d2"
-					(reference "#PWR032")
-					(unit 1)
-				)
-			)
-		)
-	)
-	(symbol
 		(lib_id "Device:C")
 		(at 177.8 130.81 0)
@@
 	)
 	(symbol
-		(lib_id "Connector:Screw_Terminal_01x04")
-		(at 232.41 83.82 180)
-		(unit 1)
-		(body_style 1)
-		(exclude_from_sim no)
-		(in_bom yes)
-		(on_board yes)
-		(in_pos_files yes)
-		(dnp no)
-		(fields_autoplaced yes)
-		(property "Reference" "J2"
-			(at 232.41 72.39 0)
-			(show_name no)
-			(do_not_autoplace no)
-			(effects
-				(font
-					(size 1.27 1.27)
-				)
-			)
-		)
-		(property "Value" "CONTACTS"
-			(at 232.41 74.93 0)
-			(show_name no)
-			(do_not_autoplace no)
-			(effects
-				(font
-					(size 1.27 1.27)
-				)
-			)
-		)
-		(property "Footprint" "Connector_PinHeader_2.54mm:PinHeader_1x04_P2.54mm_Vertical"
-			(at 232.41 83.82 0)
-			(hide yes)
-			(show_name no)
-			(do_not_autoplace no)
-			(effects
-				(font
-					(size 1.27 1.27)
-				)
-			)
-		)
-		(property "Datasheet" ""
-			(at 232.41 83.82 0)
-			(hide yes)
-			(show_name no)
-			(do_not_autoplace no)
-			(effects
-				(font
-					(size 1.27 1.27)
-				)
-			)
-		)
-		(property "Description" "Generic screw terminal, single row, 01x04, script generated (kicad-library-utils/schlib/autogen/connector/)"
-			(at 232.41 83.82 0)
-			(hide yes)
-			(show_name no)
-			(do_not_autoplace no)
-			(effects
-				(font
-					(size 1.27 1.27)
-				)
-			)
-		)
-		(pin "1"
-		)
-		(pin "2"
-		)
-		(pin "3"
-		)
-		(pin "4"
-		)
-		(instances
-			(project "Music-player"
-				(path "/f98d3056-e9c6-4dc5-a080-338d8b2650d2"
-					(reference "J2")
-					(unit 1)
-				)
-			)
-		)
-	)
-	(symbol
 		(lib_id "Device:R")
 		(at 361.95 114.3 0)
@@
 					(unit 1)
 				)
+			)
+		)
+	)
+	(symbol
+		(lib_id "Connector:Screw_Terminal_01x03")
+		(at 232.41 81.28 180)
+		(unit 1)
+		(body_style 1)
+		(exclude_from_sim no)
+		(in_bom yes)
+		(on_board yes)
+		(in_pos_files yes)
+		(dnp no)
+		(fields_autoplaced yes)
+		(property "Reference" "J2"
+			(at 232.41 72.39 0)
+			(show_name no)
+			(do_not_autoplace no)
+			(effects
+				(font
+					(size 1.27 1.27)
+				)
+			)
+		)
+		(property "Value" "Screw_Terminal_01x03"
+			(at 232.41 74.93 0)
+			(show_name no)
+			(do_not_autoplace no)
+			(effects
+				(font
+					(size 1.27 1.27)
+				)
+			)
+		)
+		(property "Footprint" "Connector_PinHeader_2.54mm:PinHeader_1x03_P2.54mm_Vertical"
+			(at 232.41 81.28 0)
+			(hide yes)
+			(show_name no)
+			(do_not_autoplace no)
+			(effects
+				(font
+					(size 1.27 1.27)
+				)
+			)
+		)
+		(property "Datasheet" ""
+			(at 232.41 81.28 0)
+			(hide yes)
+			(show_name no)
+			(do_not_autoplace no)
+			(effects
+				(font
+					(size 1.27 1.27)
+				)
+			)
+		)
+		(property "Description" "Generic screw terminal, single row, 01x03, script generated (kicad-library-utils/schlib/autogen/connector/)"
+			(at 232.41 81.28 0)
+			(hide yes)
+			(show_name no)
+			(do_not_autoplace no)
+			(effects
+				(font
+					(size 1.27 1.27)
+				)
+			)
+		)
+		(pin "3"
+		)
+		(pin "1"
+		)
+		(pin "2"
+		)
+		(instances
+			(project "Music-player"
+				(path "/f98d3056-e9c6-4dc5-a080-338d8b2650d2"
+					(reference "J2")
+					(unit 1)
+				)

Commit message: Add files via upload
Parts:
- removed C25: 1u, Capacitor_SMD:C_0402_1005Metric, symbol Device:C
- removed C29, C30, C31, C32, C33, C34, C35: 100n, Capacitor_SMD:C_0402_1005Metric, symbol Device:C
- removed R3: 10K, Resistor_SMD:R_0402_1005Metric, symbol Device:R
- added C60: 100n, Capacitor_SMD:C_0402_1005Metric, symbol Device:C
- added FB2: TDK MPZ1608S221ATA00, myotherkicadfootprintlibrary:IND_1608_TDK, symbol Device:FerriteBead
- C1: value 10u -> 1u; footprint Capacitor_SMD:C_0603_1608Metric -> Capacitor_SMD:C_0402_1005Metric
- C2: value 10u -> 2.2u; footprint Capacitor_SMD:C_0603_1608Metric -> Capacitor_SMD:C_0402_1005Metric
- FB1: footprint Resistor_SMD:R_0603_1608Metric -> myotherkicadfootprintlibrary:IND_1608_TDK
Connections:
- net GND: now also SW1.2, C60.2, FB2.2; no longer SW1.1
- net GNDA: now also FB2.1
- net RESET: now also C38.1, SW1.1
- net USB_POWER: now also C60.1
- net VDD: no longer C38.1
Other:
- note added: "C36-37 MSD_4_A"
- note removed: "C29-32 BUTTONS"
- note removed: "C33 EC11 SELECT"
- note removed: "C34 EC11_A"
- note removed: "C35 EC11_B"
- note removed: "C36 MSD_4_A"
- note removed: "C37-C38 MSD-4-A"
- moved on the sheet: C26, C27, C28, C36, C37, C38, C56, C57, C58, C59, SW1, Y1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

Commit message: First electronics iteration
Parts:
- renumbered C55 to C15, C60 to C29, C59 to C30, C58 to C31, C57 to C32, C56 to C33, C15 to C55, D4 to D3, L5 to L4, Q2 to Q1, Q3 to Q2, R16 to R3, U8 to U7
Connections:
- no-connect marks 2 -> 32
Other:
- note added: "ANTENNA"
- note added: "NRF5340-QKAA"
- moved on the sheet: C10, C12, C13, C14, C15, C16, C17, C18, C19, C20, C21, C22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

Commit message: Add files via upload
Parts:
- J5: footprint MyFootprintLibrary:SJ-43514_CUD -> MyFootprintLibrary:CUI_SJ-43514
Connections:
- net VDDA: no longer U6.13 (EN)
- net TPA_EN: now reaches U2.B14 (P1.15)
- net TPA_EN: now also U6.13 (EN)
- no-connect marks 32 -> 31
Changed lines of the file:
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@@
 	)
 	(junction
-		(at 273.05 222.25)
-		(diameter 0)
-		(color 0 0 0 0)
-	)
-	(junction
 		(at 320.04 106.68)
 		(diameter 0)
@@
 	)
 	(junction
+		(at 288.29 229.87)
+		(diameter 0)
+		(color 0 0 0 0)
+	)
+	(junction
 		(at 74.93 168.91)
 		(diameter 0)
@@
 	)
 	(junction
-		(at 273.05 219.71)
+		(at 271.78 219.71)
 		(diameter 0)
 		(color 0 0 0 0)
@@
 	)
 	(junction
-		(at 288.29 229.87)
-		(diameter 0)
-		(color 0 0 0 0)
-	)
-	(junction
 		(at 81.28 158.75)
 		(diameter 0)
@@
 	)
 	(no_connect
-		(at 154.94 219.71)
-	)
-	(no_connect
 		(at 154.94 194.31)
 	)
@@
 	(wire
 		(pts
-			(xy 280.67 224.79) (xy 273.05 224.79)
-		)
-		(stroke
-			(width 0)
-			(type default)
-		)
-	)
-	(wire
-		(pts
 			(xy 378.46 55.88) (xy 378.46 66.04)
 		)
@@
 	(wire
 		(pts
+			(xy 154.94 219.71) (xy 166.37 219.71)
+		)
+		(stroke
+			(width 0)
+			(type default)
+		)
+	)
+	(wire
+		(pts
 			(xy 246.38 266.7) (xy 246.38 265.43)
 		)
@@
 	(wire
 		(pts
-			(xy 280.67 214.63) (xy 273.05 214.63)
+			(xy 271.78 214.63) (xy 280.67 214.63)
 		)
 		(stroke
@@
 	(wire
 		(pts
-			(xy 273.05 219.71) (xy 273.05 218.44)
+			(xy 271.78 219.71) (xy 271.78 218.44)
 		)
 		(stroke
@@
 	(wire
 		(pts
-			(xy 273.05 222.25) (xy 273.05 219.71)
+			(xy 271.78 222.25) (xy 271.78 219.71)
 		)
 		(stroke
@@
 	(wire
 		(pts
-			(xy 280.67 222.25) (xy 273.05 222.25)
+			(xy 271.78 222.25) (xy 280.67 222.25)
 		)
 		(stroke
@@
 	(wire
 		(pts
-			(xy 280.67 219.71) (xy 273.05 219.71)
+			(xy 271.78 219.71) (xy 280.67 219.71)
 		)
 		(stroke
@@
 	(wire
 		(pts
-			(xy 280.67 212.09) (xy 273.05 212.09)
+			(xy 271.78 212.09) (xy 280.67 212.09)
+		)
+		(stroke
+			(width 0)
+			(type default)
+		)
+	)
+	(wire
+		(pts
+			(xy 271.78 224.79) (xy 280.67 224.79)
 		)
 		(stroke
@@
 	(wire
 		(pts
-			(xy 273.05 229.87) (xy 288.29 229.87)
+			(xy 271.78 229.87) (xy 288.29 229.87)
 		)
 		(stroke
@@
 	(wire
 		(pts
-			(xy 273.05 224.79) (xy 273.05 222.25)
-		)
-		(stroke
-			(width 0)
-			(type default)
-		)
-	)
-	(wire
-		(pts
 			(xy 372.11 46.99) (xy 375.92 46.99)
 		)
@@
 	)
 	(label "SLEEVE"
-		(at 273.05 229.87 0)
+		(at 271.78 229.87 0)
 		(effects
 			(font
@@
 	)
 	(label "OUTL"
-		(at 273.05 214.63 0)
+		(at 271.78 214.63 0)
 		(effects
 			(font
@@
 		)
 	)
+	(label "TPA_EN"
+		(at 166.37 219.71 180)
+		(effects
+			(font
+				(size 1.27 1.27)
+			)
+			(justify right bottom)
+		)
+	)
 	(label "D-"
 		(at 375.92 41.91 180)
@@
 		)
 	)
+	(label "TPA_EN"
+		(at 271.78 224.79 0)
+		(effects
+			(font
+				(size 1.27 1.27)
+			)
+			(justify left bottom)
+		)
+	)
 	(label "XC1"
 		(at 80.01 120.65 0)
@@
 	)
 	(label "OUTR"
-		(at 273.05 212.09 0)
+		(at 271.78 212.09 0)
 		(effects
 			(font
@@
 	(symbol
 		(lib_id "power:VDDA")
-		(at 273.05 218.44 0)
+		(at 271.78 218.44 0)
 		(unit 1)
 		(body_style 1)
@@
 		(dnp no)
 		(property "Reference" "#PWR024"
-			(at 273.05 222.25 0)
+			(at 271.78 222.25 0)
 			(hide yes)
 			(show_name no)
@@
 		)
 		(property "Value" "VDDA"
-			(at 276.86 217.17 0)
+			(at 275.59 217.17 0)
 			(show_name no)
 			(do_not_autoplace no)
@@
 		)
 		(property "Footprint" ""
-			(at 273.05 218.44 0)
+			(at 271.78 218.44 0)
 			(hide yes)
 			(show_name no)
@@
 		)
 		(property "Datasheet" ""
-			(at 273.05 218.44 0)
+			(at 271.78 218.44 0)
 			(hide yes)
 			(show_name no)
@@
 		)
 		(property "Description" "Power symbol creates a global label with name \"VDDA\""
-			(at 273.05 218.44 0)
+			(at 271.78 218.44 0)
 			(hide yes)
 			(show_name no)
@@
 			)
 		)
-		(property "Footprint" "MyFootprintLibrary:SJ-43514_CUD"
+		(property "Footprint" "MyFootprintLibrary:CUI_SJ-43514"
 			(at 274.32 257.81 0)
 			(hide yes)
