File: Music-player.kicad_pcb (KiCad board)
At the start: 6 copper layers, 103 parts, among them J1 USB_C_Receptacle_USB2.0_14P, J2 Screw_Terminal_01x04, J3 Screw_Terminal_01x02, J4 MSD-4-A, J5 SJ-43514, Q2 DMG2301L, Q3 DMG2301L, SW2 PLAY/STOP, SW3 SKIP, SW4 EXIT, SW5 OPTIONS, SW6 EC11_L, SW7 POWER, U1 TVS1400DRV, U2 nRF5340-QKxx, U3 SPX3819M5-L-3-3, U5 MCP73831-2-OT, U6 TPA6132A2RTE, U8 PCM5102A, Y1 Seiko SC-20S, Y2 TXC 8Q32000002

Commit message: Add files via upload
Parts:
- removed U1: TVS1400DRV, Package_SON:WSON-6-1EP_2x2mm_P0.65mm_EP1x1.6mm
- added C1: 10u, Capacitor_SMD:C_0603_1608Metric, F.Cu at (225.7, 79.0)
- added C11: 4.7u, Capacitor_SMD:C_0603_1608Metric, F.Cu at (225.7, 86.5)
- added C2: 10u, Capacitor_SMD:C_0603_1608Metric, F.Cu at (225.7, 81.5)
- added C39: 1u, Capacitor_SMD:C_0603_1608Metric, F.Cu at (225.7, 89.0)
- added C40: 1u, Capacitor_SMD:C_0603_1608Metric, F.Cu at (225.7, 91.5)
- added C41: 1u, Capacitor_SMD:C_0603_1608Metric, F.Cu at (229.7, 79.0)
- added C42: 100n, Capacitor_SMD:C_0603_1608Metric, F.Cu at (229.7, 81.5)
- added C43: 1u, Capacitor_SMD:C_0603_1608Metric, F.Cu at (229.7, 84.0)
- added C44: 1u, Capacitor_SMD:C_0603_1608Metric, F.Cu at (229.7, 86.5)
- added C45: 1u, Capacitor_SMD:C_0603_1608Metric, F.Cu at (229.7, 89.0)
- added C46: 1u, Capacitor_SMD:C_0603_1608Metric, F.Cu at (229.7, 91.5)
- added C47: 2.2u, Capacitor_SMD:C_0603_1608Metric, F.Cu at (233.7, 79.0)
- added C48: 100n, Capacitor_SMD:C_0603_1608Metric, F.Cu at (233.7, 81.5)
- added C49: 10u, Capacitor_SMD:C_0603_1608Metric, F.Cu at (233.7, 84.0)
- added C50: 1u, Capacitor_SMD:C_0603_1608Metric, F.Cu at (233.7, 86.5)
- added C51: 100n, Capacitor_SMD:C_0603_1608Metric, F.Cu at (233.7, 89.0)
- added C52: 100n, Capacitor_SMD:C_0603_1608Metric, F.Cu at (233.7, 91.5)
- added C53: 1u, Capacitor_SMD:C_0603_1608Metric, F.Cu at (237.7, 79.0)
- added C54: 10n, Capacitor_SMD:C_0603_1608Metric, F.Cu at (237.7, 81.5)
- added C6: 4.7u, Capacitor_SMD:C_0603_1608Metric, F.Cu at (225.7, 84.0)
- added D2: PRTR5V0U2X, Package_TO_SOT_SMD:SOT-143, F.Cu at (141.4, 73.8)
- added D4: LED, LED_SMD:LED_0603_1608Metric, F.Cu at (236.5, 102.1)
- added J4: MSD-4-A, MyFootprintLibrary:CUI_MSD-4-A, F.Cu at (214.5, 87.5)
- added R10: 2k, Resistor_SMD:R_0603_1608Metric, F.Cu at (237.7, 84.0)
- added R12: 470, Resistor_SMD:R_0603_1608Metric, F.Cu at (237.7, 86.5)
- added R13: 10K, Resistor_SMD:R_0603_1608Metric, F.Cu at (237.7, 89.0)
- added R14: 10K, Resistor_SMD:R_0603_1608Metric, F.Cu at (237.7, 91.5)
- added U3: SPX3819M5-L-3-3, Package_TO_SOT_SMD:SOT-23-5, F.Cu at (226.2, 95.2)
- added U5: MCP73831-2-OT, Package_TO_SOT_SMD:SOT-23-5, F.Cu at (226.2, 99.8)
- added U6: TPA6132A2RTE, Package_DFN_QFN:WQFN-16-1EP_3x3mm_P0.5mm_EP1.6x1.6mm_ThermalVias, F.Cu at (231.8, 103.5)
- added U8: PCM5102A, Package_SO:TSSOP-20_4.4x6.5mm_P0.65mm, F.Cu at (233.6, 96.8)
- E1: value 2450AT18B100E -> 2450AT43B100E; footprint MyFootprintLibrary:XDCR_2450AT18B100E -> MyFootprintLibrary:ANTENNA_2450AT43B100E
- FB1: value BLM18PG221SN1D -> TDK MPZ1608S221ATA00
- J1: value USB_C_Receptacle_USB2.0_14P -> USB_C_Receptacle_USB2.0_16P
- moved R2 104.8 mm to (144.5, 72.8)
- moved R1 99.7 mm to (138.2, 72.8), turned to 180 degrees
- moved Q3 4.72 mm to (137.7, 75.8)
- moved C46 3.85 mm to (164.3, 108.6)
- moved FB1 3.85 mm to (147.4, 108.5)
- moved U8 3.85 mm to (146.7, 103.8)
- moved C45 3.85 mm to (165.1, 105.8)
- moved C47 3.85 mm to (165.1, 102.6)
- moved C50 3.85 mm to (159.9, 102.1)
- moved C52 3.85 mm to (144.1, 108.7)
- moved C41 3.85 mm to (141.3, 105.5)
- moved C7 3.85 mm to (150.0, 110.8)
- moved U6 3.85 mm to (161.0, 105.6)
- moved C39 3.85 mm to (151.5, 105.6)
- moved C40 3.85 mm to (153.0, 105.6)
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Connections:
- net /CHARGING renamed /VBUS
- J1 pad A8: (no net) -> GND
- J1 pad B8: (no net) -> GND
- Y2 pad 2: GND -> /XC2
- Y2 pad 3: /XC2 -> (no net)
- Y2 pad 4: GND -> (no net)
Routing:
- net /D+: track 2.11 -> 18.5 mm
- net /D-: track 2.40 -> 18.4 mm
- net /LRCK: track 11.4 -> 19.9 mm
- net /VBUS: track 31.8 -> 37.4 mm, vias 6 -> 7
- net /USB_POWER: track 24.4 -> 30.0 mm, vias 5 -> 6
- net /BCK: track 8.93 -> 12.8 mm
- net /DIN: track 10.3 -> 14.1 mm
- net Net-(J1-CC1): track 0.00 -> 2.35 mm
- net Net-(J1-CC2): track 0.00 -> 2.19 mm
- net GND: vias 37 -> 38
- removed copper zone on F.Cu, net GND
Other:
- board outline added: 50 x 50 mm

Commit message: Add files via upload
Parts:
- removed the C37 at (138.1, 93.5)
- removed the C38 at (136.5, 93.5)
- removed the C39 at (151.5, 105.6)
- removed the C40 at (153.0, 105.6)
- removed the C41 at (141.3, 105.5)
- removed the C42 at (150.4, 108.4)
- removed the C43 at (154.6, 105.5)
- removed the C44 at (156.1, 104.0)
- removed the C45 at (165.1, 105.8)
- removed the C46 at (164.3, 108.6)
- removed the C47 at (165.1, 102.6)
- removed the C48 at (151.6, 100.7)
- removed the C49 at (153.1, 100.7)
- removed the C50 at (159.9, 102.1)
- removed the C51 at (159.9, 100.2)
- removed the C52 at (144.1, 108.7)
- removed the C53 at (141.9, 108.0)
- removed C7: 100n, Capacitor_SMD:C_0603_1608Metric
- removed C8: 1u, Capacitor_SMD:C_0603_1608Metric
- removed FB1: TDK MPZ1608S221ATA00, Resistor_SMD:R_0603_1608Metric
- removed the J4 at (127.0, 95.5)
- removed the R13 at (138.1, 88.0)
- removed the R14 at (140.1, 91.9)
- removed SW6: EC11_L, Rotary_Encoder:RotaryEncoder_Alps_EC11E-Switch_Vertical_H20mm_MountingHoles
- removed the U6 at (161.0, 105.6)
- removed the U8 at (146.7, 103.8)
- added REF**: MountingHole_2.2mm_M2, MountingHole:MountingHole_2.2mm_M2, F.Cu at (124.4, 64.7)
- added REF**: MountingHole_2.2mm_M2, MountingHole:MountingHole_2.2mm_M2, F.Cu at (164.9, 106.7)
- C10, C12, C13, C14, C16, C17, C18, C19, C20, C21, C22, C23, C24, C25, C28, C29, C3, C30, C31, C32, C33, C34, C35, C36, C38, C39, C4, C40, C41, C42, C43, C44, C45, C46, C47, C48, C50, C51, C52, C53, C54: footprint Capacitor_SMD:C_0603_1608Metric -> Capacitor_SMD:C_0402_1005Metric
- L1, L2, L3: footprint Inductor_SMD:L_0201_0603Metric -> Inductor_SMD:L_0603_1608Metric
- R1, R10, R11, R12, R13, R14, R15, R16, R18, R2, R3, R4, R5, R6, R7, R8, R9: footprint Resistor_SMD:R_0603_1608Metric -> Resistor_SMD:R_0402_1005Metric
- moved C13 130.8 mm to (150.8, 76.4)
- moved C12 125.1 mm to (150.8, 75.2)
- moved C10 123.0 mm to (147.2, 76.2), turned to 180 degrees
- moved C1 120.7 mm to (105.3, 87.9)
- moved C2 120.7 mm to (105.3, 90.4)
- moved C6 120.7 mm to (105.3, 92.9)
- moved C37 118.8 mm to (139.3, 86.6), turned to -90 degrees
- moved C38 116.0 mm to (137.9, 86.0), turned to -90 degrees
- moved R4 106.5 mm to (147.2, 75.0), turned to 180 degrees
- moved R13 100.8 mm to (137.3, 79.6), turned to 90 degrees
- moved R14 100.0 mm to (138.4, 79.6), turned to 90 degrees
- moved C47 93.0 mm to (142.4, 96.8), turned to -90 degrees
- moved C51 90.4 mm to (143.7, 97.9), turned to -90 degrees
- moved C50 89.4 mm to (145.0, 97.9), turned to -90 degrees
- moved C45 87.3 mm to (142.5, 94.4), turned to 90 degrees
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Routing:
- net /MSD_CS: track 15.8 -> 1.31 mm, vias 2 -> 1
- net /BCK: track 12.8 -> 24.3 mm
- net /MOSI: track 12.3 -> 2.68 mm
- net /DIN: track 14.1 -> 23.3 mm
- net VDDA: track 26.4 -> 19.9 mm, vias 9 -> 6
- net /RF: track 15.7 -> 20.7 mm
- net /MISO: track 10.4 -> 15.3 mm, vias 0 -> 2
- net /XC1: track 4.33 -> 0.00 mm
- net Net-(U2-DECD): track 0.00 -> 4.24 mm
- net Net-(U2-DECUSB): track 3.32 -> 7.02 mm
- net GND: track 8.89 -> 12.5 mm, vias 38 -> 41
- net /TIP: track 0.00 -> 3.57 mm, vias 0 -> 1
- net /CD: track 10.5 -> 13.8 mm, vias 0 -> 2
- net /RING_1: track 0.00 -> 3.13 mm, vias 0 -> 1
- net GNDA: track 8.69 -> 11.8 mm
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Other:
- board text removed: "C44"

Commit message: Add files via upload
Parts:
- removed SW2: PLAY/STOP, MyFootprintLibrary:SW_K2-1107ST-A4DW-06_HRO
- removed SW3: SKIP, MyFootprintLibrary:SW_K2-1107ST-A4DW-06_HRO
- removed SW4: EXIT, MyFootprintLibrary:SW_K2-1107ST-A4DW-06_HRO
- removed SW5: OPTIONS, MyFootprintLibrary:SW_K2-1107ST-A4DW-06_HRO
- removed SW7: POWER, MyFootprintLibrary:SW_K2-1107ST-A4DW-06_HRO
- added C7: 100n, Capacitor_SMD:C_0402_1005Metric, F.Cu at (198.9, 80.1)
- added C8: 1u, Capacitor_SMD:C_0402_1005Metric, F.Cu at (198.9, 82.1)
- added FB1: TDK MPZ1608S221ATA00, Resistor_SMD:R_0603_1608Metric, F.Cu at (195.4, 80.4)
- added SW1: RESET, myotherkicadfootprintlibrary:B3U-1000P, F.Cu at (190.5, 82.5)
- added SW6: EC11_L, Rotary_Encoder:RotaryEncoder_Alps_EC11E-Switch_Vertical_H20mm_MountingHoles, F.Cu at (188.3, 69.0)
- Y2: footprint MyFootprintLibrary:XTAL_8Q-32.000MEEV-T -> myotherkicadfootprintlibrary:XTAL_8Q-32.000MEEV-T
- moved D4 62.8 mm to (294.0, 132.2)
- moved U5 62.8 mm to (279.4, 132.9)
- moved C11 62.8 mm to (285.0, 130.6)
- moved C6 62.8 mm to (158.5, 126.2)
- moved R10 62.8 mm to (290.9, 117.3)
- moved R12 62.8 mm to (284.0, 134.2)
- moved C1 46.5 mm to (143.7, 114.1)
- moved C2 46.5 mm to (143.7, 116.6)
- moved U3 46.5 mm to (264.6, 121.4)
- moved C54 46.5 mm to (276.1, 107.7)
- moved REF** 42.0 mm to (122.9, 106.7), turned to 90 degrees
- moved REF** 42.0 mm to (164.9, 64.7), turned to 90 degrees
- moved U4 37.1 mm to (135.0, 65.5)
- moved E1 36.9 mm to (166.7, 105.7), turned to 90 degrees
- moved D4 31.3 mm to (158.4, 72.7), turned to 90 degrees
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Connections:
- U2 pad A17: /EC11_A -> /DC
- U2 pad AL21: /DC -> /RES
- U2 pad U31: /RES -> /EC11_A
- Y2 pad 1: /XC1 -> /XC2
- Y2 pad 2: /XC2 -> GND
- Y2 pad 3: (no net) -> /XC1
- Y2 pad 4: (no net) -> GND
Routing:
- net /MOSI: track 2.68 -> 41.1 mm
- net /RES: track 0.00 -> 32.3 mm, vias 0 -> 1
- net /SST_CS: track 0.00 -> 31.5 mm, vias 0 -> 1
- net /BLK: track 0.00 -> 30.2 mm, vias 0 -> 1
- net /SCK: track 11.1 -> 40.0 mm, vias 2 -> 3
- net /DC: track 0.00 -> 18.9 mm, vias 0 -> 1
- net /MSD_CS: track 1.31 -> 17.1 mm, vias 1 -> 2
- net /TIP: track 3.57 -> 18.2 mm
- net /D-: track 16.3 -> 30.9 mm, vias 1 -> 0
- net /D+: track 16.3 -> 29.7 mm, vias 1 -> 0
- net Net-(U2-DECR): track 2.11 -> 13.7 mm, vias 0 -> 2
- net /LRCK: track 22.5 -> 13.2 mm, vias 0 -> 2
- net /DIN: track 23.3 -> 14.1 mm, vias 0 -> 2
- net /BCK: track 24.3 -> 15.3 mm, vias 0 -> 2
- net GND: track 12.5 -> 20.3 mm, vias 41 -> 34
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- removed copper zone on In1.Cu, net GND
Other:
- board text added: "GET ANOTHER FOOTPRINT FOR THE CRYSTAL"

Commit message: Add files via upload
Parts:
- removed the C1 at (143.7, 114.1)
- removed the C11 at (285.0, 130.6)
- removed the C2 at (143.7, 116.6)
- removed C20, C21, C23, C28, C29, C30, C31, C32, C33, C34, C35, C36, C7: 100n, Capacitor_SMD:C_0402_1005Metric
- removed C24, C25, C4, C8: 1u, Capacitor_SMD:C_0402_1005Metric
- removed C5: 4.7u, Capacitor_SMD:C_0603_1608Metric
- removed the C54 at (276.1, 107.7)
- removed the C6 at (158.5, 126.2)
- removed D1: POWER, LED_SMD:LED_0603_1608Metric
- removed the D4 at (294.0, 132.2)
- removed FB1: TDK MPZ1608S221ATA00, Resistor_SMD:R_0603_1608Metric
- removed J2: Screw_Terminal_01x04, TerminalBlock_Phoenix:TerminalBlock_Phoenix_PT-1,5-4-3.5-H_1x04_P3.50mm_Horizontal
- removed L1: 10uH, Inductor_SMD:L_0603_1608Metric
- removed the R10 at (290.9, 117.3)
- removed R11: 22k, Resistor_SMD:R_0402_1005Metric
- removed the R12 at (284.0, 134.2)
- removed R15: 4.7k, Resistor_SMD:R_0402_1005Metric
- removed R16: 10k, Resistor_SMD:R_0402_1005Metric
- removed R18: 47K, Resistor_SMD:R_0402_1005Metric
- removed R3: 10K, Resistor_SMD:R_0402_1005Metric
- removed R5: 100, Resistor_SMD:R_0402_1005Metric
- removed R6: 1k, Resistor_SMD:R_0402_1005Metric
- removed R7: 2.2k, Resistor_SMD:R_0402_1005Metric
- removed R8, R9: 1M, Resistor_SMD:R_0402_1005Metric
- removed SW1: RESET, myotherkicadfootprintlibrary:B3U-1000P
- removed SW6: EC11_L, Rotary_Encoder:RotaryEncoder_Alps_EC11E-Switch_Vertical_H20mm_MountingHoles
- removed the U3 at (264.6, 121.4)
- removed the U5 at (279.4, 132.9)
- C15: footprint Capacitor_SMD:C_0603_1608Metric -> Capacitor_SMD:C_0402_1005Metric
- L2, L3: footprint Inductor_SMD:L_0603_1608Metric -> Inductor_SMD:L_0402_1005Metric
- Y2: value TXC 8Q32000002 -> NX2016SA-CS06654; footprint myotherkicadfootprintlibrary:XTAL_8Q-32.000MEEV-T -> MyFootprintLibrary:NX2016SA_NDK
- moved C15 139.1 mm to (158.0, 85.8), turned to -90 degrees
- moved C13 5.59 mm to (154.5, 83.1)
- moved R4 5.25 mm to (147.2, 72.5)
- moved L3 4.84 mm to (149.4, 81.3), turned to 180 degrees
- moved C10 2.61 mm to (149.4, 80.3), turned to 0 degrees
- moved C3 2.55 mm to (146.6, 80.9)
- moved C42 2.20 mm to (146.5, 97.4)
- moved C37 1.87 mm to (136.9, 83.0)
- moved C39 1.85 mm to (147.0, 98.8)
- moved C41 1.85 mm to (156.3, 99.0)
- moved C48 1.85 mm to (146.8, 102.5)
- moved C40 1.85 mm to (146.5, 100.2)
- moved C43 1.85 mm to (143.2, 100.4)
- moved C44 1.85 mm to (143.2, 101.7)
- moved C45 1.85 mm to (137.0, 100.8)
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Connections:
- U2 pad A17: /DC -> /BLK
- U2 pad AL21: /RES -> /SST_CS
- U2 pad AL23: /SST_CS -> /DC
- U2 pad AL27: /BLK -> /RES
Routing:
- net /DC: track 18.9 -> 47.4 mm
- net /RES: track 32.3 -> 51.6 mm
- net GND: track 20.3 -> 38.6 mm, vias 34 -> 40
- net /CD: track 7.39 -> 20.7 mm, vias 3 -> 1
- net /SST_CS: track 31.5 -> 44.6 mm
- net /BLK: track 30.2 -> 20.2 mm
- net /SCK: track 40.0 -> 33.9 mm, vias 3 -> 2
- net Net-(U2-DECUSB): track 7.42 -> 12.7 mm
- net /VBUS: track 37.2 -> 41.6 mm, vias 6 -> 5
- net VDD: track 33.8 -> 38.0 mm, vias 28 -> 29
- net /MOSI: track 41.1 -> 37.9 mm
- net /DIN: track 14.1 -> 15.9 mm
- net /BCK: track 15.3 -> 17.2 mm
- net /LRCK: track 13.2 -> 15.0 mm
- net /USB_POWER: track 27.3 -> 29.0 mm, vias 2 -> 4
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- added copper zone on In1.Cu, net GND

Commit message: Add files via upload
Parts:
- added C1: 10u, Capacitor_SMD:C_0603_1608Metric, F.Cu at (223.8, 60.8)
- added C11: 4.7u, Capacitor_SMD:C_0603_1608Metric, F.Cu at (223.8, 70.8)
- added C2: 10u, Capacitor_SMD:C_0603_1608Metric, F.Cu at (223.8, 63.3)
- added C20: 100n, Capacitor_SMD:C_0402_1005Metric, F.Cu at (204.7, 81.7)
- added C21: 100n, Capacitor_SMD:C_0402_1005Metric, F.Cu at (204.7, 83.7)
- added C23: 100n, Capacitor_SMD:C_0402_1005Metric, F.Cu at (204.7, 85.6)
- added C24: 1u, Capacitor_SMD:C_0402_1005Metric, F.Cu at (204.7, 87.6)
- added C25: 1u, Capacitor_SMD:C_0402_1005Metric, F.Cu at (207.6, 75.8)
- added C28: 100n, Capacitor_SMD:C_0402_1005Metric, F.Cu at (207.6, 77.8)
- added C29: 100n, Capacitor_SMD:C_0402_1005Metric, F.Cu at (207.6, 79.7)
- added C30: 100n, Capacitor_SMD:C_0402_1005Metric, F.Cu at (207.6, 81.7)
- added C31: 100n, Capacitor_SMD:C_0402_1005Metric, F.Cu at (207.6, 83.7)
- added C32: 100n, Capacitor_SMD:C_0402_1005Metric, F.Cu at (207.6, 85.6)
- added C33: 100n, Capacitor_SMD:C_0402_1005Metric, F.Cu at (207.6, 87.6)
- added C34: 100n, Capacitor_SMD:C_0402_1005Metric, F.Cu at (210.4, 75.8)
- added C35: 100n, Capacitor_SMD:C_0402_1005Metric, F.Cu at (210.4, 77.8)
- added C36: 100n, Capacitor_SMD:C_0402_1005Metric, F.Cu at (210.4, 79.7)
- added C4: 1u, Capacitor_SMD:C_0402_1005Metric, F.Cu at (204.7, 75.8)
- added C5: 4.7u, Capacitor_SMD:C_0603_1608Metric, F.Cu at (223.8, 65.8)
- added C54: 10n, Capacitor_SMD:C_0402_1005Metric, F.Cu at (210.4, 81.7)
- added C6: 4.7u, Capacitor_SMD:C_0603_1608Metric, F.Cu at (223.8, 68.3)
- added C7: 100n, Capacitor_SMD:C_0402_1005Metric, F.Cu at (204.7, 77.8)
- added C8: 1u, Capacitor_SMD:C_0402_1005Metric, F.Cu at (204.7, 79.7)
- added D1: POWER, LED_SMD:LED_0603_1608Metric, F.Cu at (197.1, 85.8)
- added D4: LED, LED_SMD:LED_0603_1608Metric, F.Cu at (197.1, 88.3)
- added FB1: TDK MPZ1608S221ATA00, Resistor_SMD:R_0603_1608Metric, F.Cu at (223.8, 73.4)
- added J2: Screw_Terminal_01x04, TerminalBlock_Phoenix:TerminalBlock_Phoenix_PT-1,5-4-3.5-H_1x04_P3.50mm_Horizontal, F.Cu at (214.6, 78.9)
- added L1: 10uH, Inductor_SMD:L_0402_1005Metric, F.Cu at (213.3, 85.7)
- added R10: 2k, Resistor_SMD:R_0402_1005Metric, F.Cu at (216.2, 91.7)
- added R11: 22k, Resistor_SMD:R_0402_1005Metric, F.Cu at (151.6, 105.0)
- added R12: 470, Resistor_SMD:R_0402_1005Metric, F.Cu at (219.1, 87.7)
- added R15: 4.7k, Resistor_SMD:R_0402_1005Metric, F.Cu at (146.5, 105.0)
- added R16: 10k, Resistor_SMD:R_0402_1005Metric, F.Cu at (149.0, 105.0)
- added R3: 10K, Resistor_SMD:R_0402_1005Metric, F.Cu at (213.3, 87.7)
- added R5: 100, Resistor_SMD:R_0402_1005Metric, F.Cu at (213.3, 89.7)
- added R6: 1k, Resistor_SMD:R_0402_1005Metric, F.Cu at (141.4, 105.0)
- added R7: 2.2k, Resistor_SMD:R_0402_1005Metric, F.Cu at (143.9, 105.0)
- added R8: 1M, Resistor_SMD:R_0402_1005Metric, F.Cu at (216.2, 87.7)
- added R9: 1M, Resistor_SMD:R_0402_1005Metric, F.Cu at (216.2, 89.7)
- added SW1: RESET, myotherkicadfootprintlibrary:B3U-1000P, F.Cu at (224.8, 88.0)
- added U1: ~, Connector_PinHeader_2.54mm:PinHeader_1x09_P2.54mm_Vertical, F.Cu at (133.8, 108.2)
- added U3: SPX3819M5-L-3-3, Package_TO_SOT_SMD:SOT-23-5, F.Cu at (192.5, 86.9)
- added U5: MCP73831-2-OT, Package_TO_SOT_SMD:SOT-23-5, F.Cu at (192.5, 91.5)
Connections:
- U2 pad AE31: /BUTTONS -> /BTN
- U2 pad AL19: /EC11_B -> /ENCA
- U2 pad U31: /EC11_A -> /ENCB
Routing:
- net /ENCB: track 0.00 -> 31.0 mm, vias 0 -> 1
- net /ENCA: track 0.00 -> 28.7 mm
- net /BTN: track 0.00 -> 28.6 mm, vias 0 -> 2
- net VDD: track 38.0 -> 55.5 mm, vias 29 -> 28
- net Net-(U1-SW3): track 0.00 -> 2.70 mm
- net Net-(U1-SW2): track 0.00 -> 2.70 mm
- net Net-(U1-SW1): track 0.00 -> 2.69 mm
- net Net-(U1-SW4): track 0.00 -> 2.69 mm
- net Net-(U1-SW5): track 0.00 -> 2.69 mm
- net /EC11_A: track 1.81 -> 0.00 mm, vias 1 -> 0
- net /D+: track 29.8 -> 28.2 mm
- net /RES: track 51.6 -> 50.5 mm
- net GNDA: track 11.5 -> 10.8 mm
- net GND: track 38.6 -> 39.2 mm
- net Net-(D4-K): track 3.26 -> 2.73 mm
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
Commit message: Add files via upload
Parts:
- removed the U3 at (138.9, 71.9)
- removed the U5 at (155.7, 71.5)
- moved C20 62.3 mm to (142.7, 88.3), turned to 180 degrees
- moved C4 58.3 mm to (146.6, 80.9), turned to 90 degrees
- moved U3 55.6 mm to (138.9, 71.9), turned to 180 degrees
- moved C23 54.9 mm to (150.2, 91.8), turned to -90 degrees
- moved C21 51.3 mm to (153.5, 87.8)
- moved U5 41.9 mm to (155.7, 71.5), turned to 180 degrees
- moved J2 20.0 mm to (196.7, 70.1)
- moved C22 11.9 mm to (142.7, 89.3), turned to 180 degrees
- moved C16 9.79 mm to (144.2, 84.0), turned to 90 degrees
- moved C19 8.21 mm to (144.3, 90.4), turned to 180 degrees
- moved C18 5.62 mm to (148.4, 90.6)
- moved C12 3.26 mm to (151.8, 80.8), turned to 90 degrees
- moved C3 2.86 mm to (149.4, 81.3), turned to 180 degrees
- moved L3 1.52 mm to (150.9, 80.8), turned to 90 degrees
- moved Y2 1.35 mm to (153.9, 81.0), turned to 0 degrees
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Connections:
- C3 pad 1: Net-(U2-DECA) -> Net-(U2-DECN)
- U2 pad A23: Net-(U2-DECA) -> Net-(U2-DECN)
Routing:
- net VDD: track 55.5 -> 44.3 mm, vias 28 -> 25
- net Net-(U2-DECR): track 13.0 -> 6.44 mm, vias 3 -> 1
- net GND: track 39.2 -> 34.1 mm, vias 40 -> 41
- net /XC1: track 4.68 -> 0.00 mm
- net Net-(U2-DECA): track 6.14 -> 2.86 mm
- net /XC2: track 2.76 -> 0.00 mm
- net Net-(U2-DECN): track 0.00 -> 1.96 mm
- net /MOSI: track 37.9 -> 36.1 mm
- net /D+: track 28.2 -> 29.8 mm
- net /D-: track 30.9 -> 32.5 mm
- net /ENCA: track 28.7 -> 30.2 mm, vias 0 -> 2
- net /CD: track 20.7 -> 20.1 mm
- net /MSD_CS: track 17.0 -> 16.4 mm
- net /DC: track 47.4 -> 46.8 mm
- net GNDA: track 10.8 -> 10.3 mm, vias 14 -> 13

Commit message: Add files via upload
Parts:
- added C55: 100n, Capacitor_SMD:C_0402_1005Metric, F.Cu at (147.2, 91.7)
- J2: value Screw_Terminal_01x04 -> CONTACTS; footprint TerminalBlock_Phoenix:TerminalBlock_Phoenix_PT-1,5-4-3.5-H_1x04_P3.50mm_Horizontal -> Connector_PinHeader_2.54mm:PinHeader_1x04_P2.54mm_Vertical
- moved J2 21.0 mm to (176.1, 74.3)
- moved C22 1.26 mm to (142.3, 88.1)
- moved C10 1.10 mm to (149.4, 79.2)
- moved C20 0.98 mm to (142.3, 89.2)
- moved C18 0.93 mm to (149.0, 91.3), turned to 0 degrees
- moved C23 0.85 mm to (151.0, 91.8)
- moved C3 0.66 mm to (149.9, 80.8), turned to 90 degrees
Routing:
- net VDD: track 44.3 -> 47.9 mm
- net /SST_CS: track 44.4 -> 45.5 mm
- net Net-(U2-DECD): track 3.74 -> 4.72 mm
- net /ENCA: track 30.2 -> 29.3 mm, vias 2 -> 0
- net /RES: track 50.5 -> 51.3 mm
- net /DC: track 46.8 -> 47.6 mm
- net GNDA: track 10.3 -> 9.82 mm, vias 13 -> 12
- net GND: vias 41 -> 42

Commit message: Add files via upload
Parts:
- added C56: 100n, Capacitor_SMD:C_0402_1005Metric, F.Cu at (146.4, 80.8)
- added C57: 100n, Capacitor_SMD:C_0402_1005Metric, F.Cu at (148.9, 80.7)
- added C58: 100n, Capacitor_SMD:C_0402_1005Metric, F.Cu at (151.9, 80.7)
- added C59: 100n, Capacitor_SMD:C_0402_1005Metric, F.Cu at (154.2, 82.7)
- Y2: footprint MyFootprintLibrary:NX2016SA_NDK -> myotherkicadfootprintlibrary:NX2016SA_NDK
- moved C12 1.63 mm to (151.3, 79.3), turned to 180 degrees
- moved C4 1.50 mm to (147.1, 79.5), turned to 0 degrees
- moved C16 1.31 mm to (143.2, 83.2)
- moved Y2 1.20 mm to (154.9, 80.3)
- moved C13 1.10 mm to (155.6, 83.1)
- moved C19 0.94 mm to (144.2, 91.3)
- moved C3 0.15 mm to (149.9, 80.7)
- moved L3 0.15 mm to (150.9, 80.7)
- moved C10 0.12 mm to (149.4, 79.3)
- moved C21 0.07 mm to (153.6, 87.8)
Routing:
- net VDD: track 47.9 -> 57.6 mm, vias 25 -> 26
- net Net-(U2-DECR): track 6.44 -> 14.2 mm, vias 1 -> 2
- net /XC2: track 0.00 -> 5.31 mm
- net /XC1: track 0.00 -> 5.17 mm
- net /MSD_CS: track 16.4 -> 18.3 mm
- net Net-(U2-DECA): track 2.86 -> 4.04 mm
- net Net-(U2-DECD): track 4.72 -> 5.12 mm, vias 2 -> 0
- net GND: vias 42 -> 48
