File: Music-player.kicad_pcb (KiCad board)
At the start: 6 copper layers, 50 x 50 mm, 111 parts, among them J1 USB_C_Receptacle_USB2.0_16P, J2 CONTACTS, J3 Screw_Terminal_01x02, J4 MSD-4-A, J5 SJ-43514, Q2 DMG2301L, Q3 DMG2301L, SW1 RESET, U2 nRF5340-QKxx, U3 SPX3819M5-L-3-3, U5 MCP73831-2-OT, U6 TPA6132A2RTE, U8 PCM5102A, Y1 Seiko SC-20S, Y2 NX2016SA-CS06654

Commit message: Add files via upload
Parts:
- removed the C1 at (223.8, 60.8)
- removed the C11 at (223.8, 70.8)
- removed the C2 at (223.8, 63.3)
- removed the C54 at (136.9, 69.3)
- removed the C54 at (210.4, 81.7)
- removed the C6 at (223.8, 68.3)
- removed the D4 at (197.1, 88.3)
- removed the R10 at (216.2, 91.7)
- removed the R10 at (152.2, 73.2)
- removed the R12 at (219.1, 87.7)
- removed the R12 at (156.2, 74.9)
- removed SW1: RESET, myotherkicadfootprintlibrary:B3U-1000P
- added C54: 10n, Capacitor_SMD:C_0402_1005Metric, F.Cu at (136.9, 69.3)
- added R10: 2k, Resistor_SMD:R_0402_1005Metric, F.Cu at (152.2, 72.9)
- added R12: 470, Resistor_SMD:R_0402_1005Metric, F.Cu at (156.7, 74.4)
- J2: value CONTACTS -> Screw_Terminal_01x03; footprint Connector_PinHeader_2.54mm:PinHeader_1x04_P2.54mm_Vertical -> Connector_PinHeader_2.54mm:PinHeader_1x03_P2.54mm_Vertical
- moved C38 122.5 mm to (247.3, 29.8), turned to 0 degrees
- moved C31 97.3 mm to (278.5, 17.1)
- moved C32 97.3 mm to (278.8, 19.3)
- moved C34 94.6 mm to (281.6, 13.4)
- moved C35 94.6 mm to (281.6, 15.4)
- moved R8 75.7 mm to (142.1, 72.8)
- moved R9 74.2 mm to (143.9, 72.8)
- moved C36 74.0 mm to (136.4, 81.8)
- moved C29 72.6 mm to (261.3, 30.9), turned to 90 degrees
- moved C30 71.8 mm to (260.0, 32.7)
- moved C28 71.2 mm to (138.0, 62.6)
- moved L1 70.7 mm to (142.7, 82.8)
- moved C33 69.1 mm to (255.3, 37.7), turned to 90 degrees
- moved C25 60.5 mm to (147.1, 78.5)
- moved C24 56.2 mm to (148.9, 80.7), turned to 90 degrees
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Connections:
- J2 pad 2: VDD -> /SWDIO
Routing:
- net /AIN0: track 0.00 -> 41.6 mm, vias 0 -> 4
- net /SWDCLK: track 0.00 -> 24.4 mm, vias 0 -> 1
- net /SWDIO: track 0.00 -> 23.6 mm, vias 0 -> 1
- net VDD: track 57.6 -> 69.9 mm, vias 26 -> 31
- net /RESET: track 0.00 -> 4.03 mm
- net Net-(U2-DCCH): track 0.00 -> 2.78 mm
- net GND: track 34.1 -> 36.4 mm, vias 48 -> 51
- net /USB_POWER: track 29.0 -> 30.6 mm
- net Net-(D1-A): track 0.00 -> 1.22 mm
- net Net-(U5-STAT): track 3.09 -> 2.30 mm
- net /ENCB: track 31.0 -> 31.6 mm

Commit message: Add files via upload
Parts:
- removed C29, C30, C31, C32, C33, C34, C35: 100n, Capacitor_SMD:C_0402_1005Metric
- removed C5: 4.7u, Capacitor_SMD:C_0603_1608Metric
- removed FB1: TDK MPZ1608S221ATA00, Resistor_SMD:R_0603_1608Metric
- removed R3: 10K, Resistor_SMD:R_0402_1005Metric
- added C60: 100n, Capacitor_SMD:C_0402_1005Metric, F.Cu at (140.3, 69.2)
- added FB2: TDK MPZ1608S221ATA00, myotherkicadfootprintlibrary:IND_1608_TDK, F.Cu at (144.1, 98.5)
- added SW1: RESET, myotherkicadfootprintlibrary:B3U-1000P, B.Cu at (157.9, 92.2)
- C1: value 10u -> 1u; footprint Capacitor_SMD:C_0603_1608Metric -> Capacitor_SMD:C_0402_1005Metric
- C2: value 10u -> 2.2u; footprint Capacitor_SMD:C_0603_1608Metric -> Capacitor_SMD:C_0402_1005Metric
- moved C38 109.0 mm to (156.5, 90.1)
- moved C8 60.9 mm to (135.2, 94.7), turned to -90 degrees
- moved C7 58.4 mm to (138.0, 94.7), turned to -90 degrees
- moved C21 7.36 mm to (154.4, 87.8)
- moved C28 5.39 mm to (137.0, 67.9), turned to 180 degrees
- moved C1 1.40 mm to (139.4, 69.2), turned to 90 degrees
- moved C2 1.17 mm to (136.2, 72.3)
- moved C16 0.21 mm to (142.7, 81.9)
Connections:
- C38 pad 1: VDD -> /RESET
Routing:
- net /RESET: track 4.03 -> 8.91 mm, vias 0 -> 1
- net VDDA: track 19.8 -> 22.6 mm, vias 8 -> 9
- net GND: track 36.4 -> 34.4 mm, vias 51 -> 60
- net /USB_POWER: track 30.6 -> 31.9 mm
- net VDD: track 69.9 -> 70.7 mm, vias 31 -> 33
- net /VBUS: vias 5 -> 7
- net GNDA: vias 12 -> 13

Commit message: First electronics iteration
Parts:
- removed C25: 1u, Capacitor_SMD:C_0402_1005Metric
- added FB1: TDK MPZ1608S221ATA00, myotherkicadfootprintlibrary:IND_1608_TDK, F.Cu at (136.6, 93.4)
- moved J4 0.06 mm to (126.2, 82.8)
Routing:
- net Net-(U2-DECR): track 14.3 -> 13.7 mm
- net GND: vias 60 -> 59

Commit message: Add files via upload
Parts:
- J5: footprint MyFootprintLibrary:SJ-43514_CUD -> MyFootprintLibrary:CUI_SJ-43514
- moved J5 4.42 mm to (123.0, 98.0), turned to 0 degrees
- moved C7 0.90 mm to (137.1, 94.8)
- moved FB1 0.90 mm to (135.7, 93.5)
- moved C8 0.90 mm to (134.3, 94.8)
- moved J1 0.49 mm to (122.6, 68.3)
- renumbered C55 to C15, C60 to C29, C59 to C30, C58 to C31, C57 to C32, C56 to C33, C15 to C55, D4 to D3, L5 to L4, Q2 to Q1, Q3 to Q2, R16 to R3, U8 to U7
Connections:
- U2 pad B12: unconnected-(U2-NC-PadB12) -> /TPA_EN
- U2 pad B14: unconnected-(U2-P1.15-PadB14) -> /TPA_EN
- U6 pad 13: VDDA -> /TPA_EN
Routing:
- net /TPA_EN: track 0.00 -> 27.5 mm, vias 0 -> 3
- net /RING_1: track 9.56 -> 13.6 mm
- net /TIP: track 19.0 -> 16.2 mm
- net GNDA: track 9.82 -> 11.7 mm, vias 13 -> 14
- net VDDA: track 22.6 -> 22.1 mm
- net VDD: track 70.7 -> 70.9 mm, vias 33 -> 31
Other:
- board text removed: "U3"

Commit message: Add files via upload
Other:
- board text removed: "GET ANOTHER FOOTPRINT FOR THE CRYSTAL"
Changed lines of the file:
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@@
-		)
-	)
-	(gr_text "GET ANOTHER FOOTPRINT \nFOR THE CRYSTAL\n"
-		(at 152.65 80.8625 0)
-		(layer "Cmts.User")
-		(effects
-			(font
-				(size 1 1)
-				(thickness 0.2)
-				(bold yes)
-			)
-			(justify left bottom)
 		)
 	)

Commit message: Add files via upload
Parts:
- moved J5 2.56 mm to (125.6, 98.2)
Routing:
- net /RING_1: track 13.6 -> 10.5 mm
- net /TIP: track 16.2 -> 13.0 mm
Other:
- board size 50 x 50 mm -> 51.5 x 50 mm

Commit message: Add files via upload
Parts:
- J2: footprint Connector_PinHeader_2.54mm:PinHeader_1x03_P2.54mm_Vertical -> Connector_JST:JST_PH_S3B-PH-K_1x03_P2.00mm_Horizontal
- U1: footprint Connector_PinHeader_2.54mm:PinHeader_1x09_P2.54mm_Vertical -> Connector_JST:JST_PH_S9B-PH-K_1x09_P2.00mm_Horizontal
- U4: footprint Connector_PinHeader_2.54mm:PinHeader_1x08_P2.54mm_Vertical -> Connector_JST:JST_PH_S8B-PH-K_1x08_P2.00mm_Horizontal
- moved U4 18.2 mm to (153.2, 65.5), turned to 180 degrees
- moved U1 3.59 mm to (137.3, 108.0), turned to 0 degrees
- moved J2 3.19 mm to (163.6, 80.7), turned to 90 degrees
- moved R6 1.95 mm to (143.3, 105.0)
- moved R7 1.45 mm to (145.3, 105.0)
- moved J3 1.40 mm to (163.6, 71.8)
- moved R15 0.85 mm to (147.3, 105.0)
- moved D1 0.68 mm to (160.6, 77.2)
- moved R5 0.68 mm to (160.1, 75.2)
- moved C49 0.56 mm to (144.7, 103.0), turned to 180 degrees
- moved R3 0.35 mm to (149.3, 105.0)
- moved R11 0.21 mm to (151.3, 105.1)
- moved R9 0.15 mm to (144.1, 72.8)
Connections:
- U2 pad B12: /TPA_EN -> unconnected-(U2-NC-PadB12)
Routing:
- net VDD: track 70.9 -> 67.0 mm, vias 31 -> 33
- net /ENCB: track 31.6 -> 29.0 mm
- net /BTN: track 28.2 -> 26.3 mm
- net /SWDCLK: track 24.1 -> 22.2 mm
- net /SWDIO: track 23.6 -> 21.9 mm
- net /MOSI: track 36.1 -> 37.7 mm
- net /USB_GATE: track 32.1 -> 33.6 mm
- net /SCK: track 33.6 -> 34.9 mm
- net /DC: track 47.6 -> 48.6 mm
- net /SST_CS: track 45.5 -> 46.2 mm
- net /ENCA: track 29.3 -> 28.6 mm
- net /BLK: track 20.2 -> 19.7 mm

Commit message: Add files via upload
Parts:
- moved U1 13.2 mm to (150.5, 108.5)
- moved E1 7.95 mm to (167.0, 97.3)
- moved R11 6.67 mm to (144.7, 104.2), turned to 180 degrees
- moved R3 4.61 mm to (144.7, 105.2), turned to 180 degrees
- moved R6 3.26 mm to (144.7, 108.0), turned to 180 degrees
- moved R15 2.81 mm to (144.7, 106.1), turned to 180 degrees
- moved R7 2.09 mm to (144.7, 107.0), turned to 180 degrees
- moved SW1 1.84 mm to (156.3, 93.0), turned to -90 degrees
Routing:
- net Net-(U1-SW5): track 2.69 -> 21.1 mm
- net Net-(U1-SW4): track 2.44 -> 18.7 mm
- net VDD: track 67.0 -> 53.0 mm, vias 33 -> 32
- net Net-(U1-SW3): track 2.44 -> 16.3 mm
- net /ENCA: track 28.6 -> 42.0 mm
- net Net-(U1-SW2): track 2.44 -> 14.4 mm
- net Net-(U1-SW1): track 2.44 -> 12.6 mm
- net /RF: track 25.9 -> 17.7 mm
- net /ENCB: track 29.0 -> 23.2 mm, vias 1 -> 2
- net /BTN: track 26.3 -> 29.1 mm
