File: Music-player.kicad_pcb (KiCad board)
At the start: 6 copper layers, 51.5 x 50 mm, 95 parts, among them J1 USB_C_Receptacle_USB2.0_16P, J2 Screw_Terminal_01x03, J3 Screw_Terminal_01x02, J4 MSD-4-A, J5 SJ-43514, Q1 DMG2301L, Q2 DMG2301L, SW1 RESET, U2 nRF5340-QKxx, U3 SPX3819M5-L-3-3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

Commit message: Add files via upload
Parts:
- moved J3 1.40 mm to (162.2, 71.7)
- moved J2 1.40 mm to (162.2, 80.6)
- moved D1 1.20 mm to (159.4, 77.2)
- moved R5 1.20 mm to (158.9, 75.2)
- moved FB2 0.80 mm to (144.8, 98.8)
Routing:
- net /USB_GATE: track 33.6 -> 32.2 mm
- net /SWDIO: track 21.9 -> 20.7 mm
- net /SWDCLK: track 22.2 -> 21.6 mm
Other:
- board size 51.5 x 50 mm -> 50 x 50 mm
Changed lines of the file:
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@@
 	(footprint "Connector_JST:JST_PH_S3B-PH-K_1x03_P2.00mm_Horizontal"
 		(layer "F.Cu")
-		(at 163.55 80.65 90)
+		(at 162.15 80.6 90)
 		(descr "JST PH series connector, S3B-PH-K (http://www.jst-mfg.com/product/pdf/eng/ePH.pdf)")
 		(tags "connector JST PH horizontal")
@@
 	(footprint "myotherkicadfootprintlibrary:IND_1608_TDK"
 		(layer "F.Cu")
-		(at 144.05 98.45 180)
+		(at 144.7722 98.8 180)
 		(tags "MPZ1608S221ATA00 ")
 		(property "Reference" "FB2"
@@
 			(polygon
 				(pts
-					(xy 144.4992 98.7992) (xy 143.6008 98.7992) (xy 143.6008 98.1008) (xy 144.4992 98.1008)
+					(xy 145.2214 99.1492) (xy 144.323 99.1492) (xy 144.323 98.4508) (xy 145.2214 98.4508)
 				)
 			)
@@
 	(footprint "Resistor_SMD:R_0402_1005Metric"
 		(layer "F.Cu")
-		(at 160.1 75.1875)
+		(at 158.9 75.1875)
 		(descr "Resistor SMD 0402 (1005 Metric), square (rectangular) end terminal, IPC-7351 nominal, (Body size source: IPC-SM-782 page 72, https://www.pcb-3d.com/wordpress/wp-content/uploads/ipc-sm-782a_amendment_1_and_2.pdf)")
 		(tags "resistor")
@@
 	(footprint "LED_SMD:LED_0603_1608Metric"
 		(layer "F.Cu")
-		(at 160.6 77.1875 90)
+		(at 159.4 77.1875 90)
 		(descr "LED SMD 0603 (1608 Metric), square (rectangular) end terminal, IPC-7351 nominal, (Body size source: http://www.tortai-tech.com/upload/download/2011102023233369053.pdf)")
 		(tags "LED")
@@
 	(footprint "Connector_JST:JST_PH_S2B-PH-K_1x02_P2.00mm_Horizontal"
 		(layer "F.Cu")
-		(at 163.55 71.8 90)
+		(at 162.15 71.7 90)
 		(descr "JST PH series connector, S2B-PH-K (http://www.jst-mfg.com/product/pdf/eng/ePH.pdf)")
 		(tags "connector JST PH horizontal")
@@
 	(gr_line
 		(start 118.9 110.65)
-		(end 170.4 110.65)
+		(end 168.9 110.65)
 		(stroke
 			(width 0.05)
@@
 	)
 	(gr_line
-		(start 170.4 60.65)
+		(start 168.9 60.65)
 		(end 118.9 60.65)
 		(stroke
@@
 	)
 	(gr_line
-		(start 170.4 110.65)
-		(end 170.4 60.65)
+		(start 168.9 110.65)
+		(end 168.9 60.65)
 		(stroke
 			(width 0.05)
@@
 	)
 	(via
-		(at 159.59 75.1875)
+		(at 158.39 75.1875)
 		(size 0.5)
 		(drill 0.3)
@@
 	)
 	(via
-		(at 143.2222 98.45)
+		(at 143.9444 98.8)
 		(size 0.5)
 		(drill 0.3)
@@
 	)
 	(via
-		(at 160.6 77.975)
+		(at 159.4 77.975)
 		(size 0.5)
 		(drill 0.3)
@@
 	)
 	(via
-		(at 144.8778 98.45)
+		(at 145.6 98.8)
 		(size 0.5)
 		(drill 0.3)
@@
 	)
 	(segment
-		(start 163.5 69.75)
-		(end 163.55 69.8)
+		(start 157.5875 69.75)
+		(end 162.1 69.75)
 		(width 0.5)
 		(layer "F.Cu")
@@
 	)
 	(segment
-		(start 156.8375 70.5)
-		(end 157.5875 69.75)
+		(start 147.25 70.1)
+		(end 148.1 70.95)
 		(width 0.5)
 		(layer "F.Cu")
@@
 	)
 	(segment
-		(start 147.25 70.1)
-		(end 148.1 70.95)
+		(start 162.1 69.75)
+		(end 162.15 69.7)
 		(width 0.5)
 		(layer "F.Cu")
@@
 	)
 	(segment
-		(start 157.5875 69.75)
-		(end 163.5 69.75)
+		(start 156.8375 70.5)
+		(end 157.5875 69.75)
 		(width 0.5)
 		(layer "F.Cu")
@@
 	)
 	(segment
-		(start 164 79.05)
-		(end 164.25 79.05)
+		(start 160.35 88.3)
+		(end 160.35 80.4)
 		(width 0.15)
 		(layer "B.Cu")
@@
 	)
 	(segment
-		(start 154.5 89.45)
-		(end 159.2 89.45)
+		(start 160.35 80.4)
+		(end 162.1 78.65)
 		(width 0.15)
 		(layer "B.Cu")
@@
 	)
 	(segment
-		(start 164.25 79.05)
-		(end 164.45 78.85)
-		(width 0.15)
-		(layer "B.Cu")
-		(net "/SWDIO")
-	)
-	(segment
-		(start 160.35 88.3)
-		(end 160.35 81.85)
-		(width 0.15)
-		(layer "B.Cu")
-		(net "/SWDIO")
-	)
-	(segment
-		(start 160.35 81.85)
-		(end 163.55 78.65)
+		(start 154.5 89.45)
+		(end 159.2 89.45)
 		(width 0.15)
 		(layer "B.Cu")
@@
 	)
 	(segment
-		(start 159.5 80.7)
-		(end 163.55 76.65)
+		(start 158.95 88.6)
+		(end 159.5 88.05)
 		(width 0.15)
 		(layer "B.Cu")
@@
 	)
 	(segment
-		(start 158.95 88.6)
-		(end 159.5 88.05)
+		(start 154.45 88.6)
+		(end 158.95 88.6)
 		(width 0.15)
 		(layer "B.Cu")
@@
 	(segment
 		(start 159.5 88.05)
-		(end 159.5 80.7)
+		(end 159.5 79.25)
 		(width 0.15)
 		(layer "B.Cu")
@@
 	)
 	(segment
-		(start 154.45 88.6)
-		(end 158.95 88.6)
+		(start 159.5 79.25)
+		(end 162.15 76.6)
 		(width 0.15)
 		(layer "B.Cu")
@@
 	)
 	(segment
-		(start 160.61 76.39)
-		(end 160.6 76.4)
+		(start 159.41 76.39)
+		(end 159.4 76.4)
 		(width 0.15)
 		(layer "F.Cu")
@@
 	)
 	(segment
-		(start 160.61 75.1875)
-		(end 160.61 76.39)
+		(start 159.41 75.1875)
+		(end 159.41 76.39)
 		(width 0.15)
 		(layer "F.Cu")

Commit message: Add files via upload
Parts:
- moved J4 1.75 mm to (124.5, 82.8)
- moved R9 0.50 mm to (144.1, 72.3), turned to 90 degrees
- moved C36 0.45 mm to (136.0, 81.8)
- moved C37 0.45 mm to (136.5, 83.0)
- moved R13 0.35 mm to (135.4, 75.2)
- moved R14 0.35 mm to (136.5, 75.2)
Routing:
- net /SCK: track 34.9 -> 39.3 mm
- net /MOSI: track 37.7 -> 41.1 mm
- net VDD: track 53.0 -> 56.0 mm, vias 32 -> 33
- net /MISO: track 21.0 -> 23.9 mm
- net /CD: track 20.1 -> 21.9 mm
- net /MSD_CS: track 18.3 -> 20.0 mm
- net /AIN0: track 41.4 -> 42.1 mm

Commit message: Add files via upload
Routing:
- net VDD: track 56.0 -> 53.3 mm
- net /MISO: track 23.9 -> 22.6 mm
Other:
- outline, holes or cut-outs redrawn
Changed lines of the file:
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@@
 	)
 	(gr_line
-		(start 118.9 60.65)
+		(start 118.9 64.65)
 		(end 118.9 95.25)
 		(stroke
@@
 		(layer "Edge.Cuts")
 	)
-	(gr_line
-		(start 118.9 95.25)
-		(end 120.6 95.25)
+	(gr_arc
+		(start 118.9 64.65)
+		(mid 120.071573 61.821573)
+		(end 122.9 60.65)
 		(stroke
 			(width 0.05)
@@
 	)
 	(gr_line
-		(start 118.9 101.25)
-		(end 118.9 110.65)
+		(start 118.9 95.25)
+		(end 120.6 95.25)
 		(stroke
 			(width 0.05)
@@
 	)
 	(gr_line
-		(start 118.9 110.65)
-		(end 168.9 110.65)
+		(start 118.9 101.25)
+		(end 118.9 106.65)
 		(stroke
 			(width 0.05)
@@
 		(layer "Edge.Cuts")
 	)
+	(gr_arc
+		(start 122.9 110.65)
+		(mid 120.071573 109.478427)
+		(end 118.9 106.65)
+		(stroke
+			(width 0.05)
+			(type default)
+		)
+		(layer "Edge.Cuts")
+	)
 	(gr_line
-		(start 168.9 60.65)
-		(end 118.9 60.65)
+		(start 122.9 110.65)
+		(end 164.9 110.65)
 		(stroke
 			(width 0.05)
@@
 	)
 	(gr_line
-		(start 168.9 110.65)
-		(end 168.9 60.65)
+		(start 164.9 60.65)
+		(end 122.9 60.65)
+		(stroke
+			(width 0.05)
+			(type default)
+		)
+		(layer "Edge.Cuts")
+	)
+	(gr_arc
+		(start 164.9 60.65)
+		(mid 167.728427 61.821573)
+		(end 168.9 64.65)
+		(stroke
+			(width 0.05)
+			(type default)
+		)
+		(layer "Edge.Cuts")
+	)
+	(gr_arc
+		(start 168.9 106.65)
+		(mid 167.728427 109.478427)
+		(end 164.9 110.65)
+		(stroke
+			(width 0.05)
+			(type default)
+		)
+		(layer "Edge.Cuts")
+	)
+	(gr_line
+		(start 168.9 106.65)
+		(end 168.9 64.65)
 		(stroke
 			(width 0.05)
@@
 	)
 	(segment
+		(start 132.25 81.8)
+		(end 135.52 81.8)
+		(width 0.15)
+		(layer "F.Cu")
+		(net "VDD")
+	)
+	(segment
 		(start 146.475 83.425)
 		(end 146.475 82.425)
@@
 	)
 	(segment
-		(start 132.25 81.8)
-		(end 134.95 81.8)
-		(width 0.15)
-		(layer "F.Cu")
-		(net "VDD")
-	)
-	(segment
 		(start 144.95 83.65)
 		(end 144.95 83.7)
@@
 	)
 	(segment
-		(start 135.52 81.8)
-		(end 132.25 81.8)
-		(width 0.15)
-		(layer "F.Cu")
-		(net "VDD")
-	)
-	(segment
 		(start 151.542893 84.1)
 		(end 151.35 84.1)
@@
 	)
 	(via
-		(at 123.34 90.6)
+		(at 121.65 90.6)
 		(size 0.5)
 		(drill 0.3)
@@
 	)
 	(via
-		(at 132.89 89.7)
+		(at 131.2 89.7)
 		(size 0.5)
 		(drill 0.3)
@@
 	)
 	(segment
-		(start 136.3 78.5)
-		(end 132.25 78.5)
-		(width 0.2)
-		(layer "In3.Cu")
-		(net "/MISO")
-	)
-	(segment
 		(start 136.5 75.72)
 		(end 136.5 78.3)
@@
 	)
 	(segment
-		(start 136.3 78.5)
-		(end 135 78.5)
-		(width 0.2)
+		(start 132.25 78.5)
+		(end 136.3 78.5)
+		(width 0.15)
 		(layer "In3.Cu")
 		(net "/MISO")

Commit message: Add files via upload
Parts:
- moved U4 5.25 mm to (158.4, 65.3)
Routing:
- net /RES: track 51.6 -> 53.9 mm
- net /BLK: track 19.7 -> 22.0 mm
- net /SCK: track 39.3 -> 41.5 mm
- net /SST_CS: track 46.2 -> 48.2 mm
- net /DC: track 48.6 -> 50.5 mm
- net /MOSI: track 41.1 -> 42.8 mm

Commit message: Add files via upload
Routing:
- net GND: vias 59 -> 62
