File: ELECTRONICS/Music-player.kicad_pcb (KiCad board)
At the start: 6 copper layers, 50 x 50 mm, 95 parts, among them J1 USB_C_Receptacle_USB2.0_16P, J2 Screw_Terminal_01x03, J3 Screw_Terminal_01x02, J4 MSD-4-A, J5 SJ-43514, Q1 DMG2301L, Q2 DMG2301L, SW1 RESET, U2 nRF5340-QKxx, U3 SPX3819M5-L-3-3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

Commit message: Add files via upload
Parts:
- moved U1 1.19 mm to (149.3, 108.2)
- moved Y2 0.28 mm to (154.9, 80.0)
Connections:
- U2 pad B12: unconnected-(U2-NC-PadB12) -> /TPA_EN
Routing:
- net Net-(U1-SW3): track 16.3 -> 15.0 mm
- net Net-(U1-SW5): track 21.1 -> 19.8 mm
- net Net-(U1-SW4): track 18.7 -> 17.4 mm
- net Net-(U1-SW2): track 14.4 -> 13.1 mm
- net /ENCA: track 42.0 -> 40.9 mm
- net Net-(U1-SW1): track 12.6 -> 11.6 mm
