File: ELECTRONICS/Music-player.kicad_pcb (KiCad board)
At the start: 6 copper layers, 50 x 50 mm, 95 parts, among them J1 USB_C_Receptacle_USB2.0_16P, J2 Screw_Terminal_01x03, J3 Screw_Terminal_01x02, J4 MSD-4-A, J5 SJ-43514, Q1 DMG2301L, Q2 DMG2301L, SW1 RESET, U2 nRF5340-QKxx, U3 SPX3819M5-L-3-3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

Commit message: Add files via upload
Parts:
- C26: footprint Capacitor_SMD:C_0603_1608Metric -> Capacitor_SMD:C_0402_1005Metric
- moved C26 0.11 mm to (141.0, 82.4)
Connections:
- U2 pad B12: /TPA_EN -> unconnected-(U2-NC-PadB12)
Routing:
- net GND: track 33.7 -> 34.5 mm
Changed lines of the file:
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@@
 		(sheetname "/")
 		(sheetfile "Music-player.kicad_sch")
+		(units
+			(unit
+				(name "A")
+				(pins "4" "2" "3" "1")
+			)
+		)
 		(attr through_hole)
 		(duplicate_pad_numbers_are_jumpers no)
@@
 		(sheetname "/")
 		(sheetfile "Music-player.kicad_sch")
+		(units
+			(unit
+				(name "A")
+				(pins "3" "9" "1" "2" "4" "5" "6" "7" "8")
+			)
+		)
 		(attr through_hole)
 		(duplicate_pad_numbers_are_jumpers no)
@@
 		)
 	)
-	(footprint "Capacitor_SMD:C_0603_1608Metric"
+	(footprint "Capacitor_SMD:C_0402_1005Metric"
 		(layer "F.Cu")
-		(at 140.95 82.3 90)
-		(descr "Capacitor SMD 0603 (1608 Metric), square (rectangular) end terminal, IPC-7351 nominal, (Body size source: IPC-SM-782 page 76, https://www.pcb-3d.com/wordpress/wp-content/uploads/ipc-sm-782a_amendment_1_and_2.pdf)")
+		(at 141 82.4 90)
+		(descr "Capacitor SMD 0402 (1005 Metric), square (rectangular) end terminal, IPC-7351 nominal, (Body size source: IPC-SM-782 page 76, https://www.pcb-3d.com/wordpress/wp-content/uploads/ipc-sm-782a_amendment_1_and_2.pdf)")
 		(tags "capacitor")
 		(property "Reference" "C26"
-			(at -3.7 0.32 90)
+			(at 0 -1.16 90)
 			(layer "F.SilkS")
-			(hide yes)
 			(effects
 				(font
@@
 		)
 		(property "Value" "2.2u"
-			(at 0 1.43 90)
+			(at 0 1.16 90)
 			(layer "F.Fab")
 			(effects
@@
 		(duplicate_pad_numbers_are_jumpers no)
 		(fp_line
-			(start -0.14058 -0.51)
-			(end 0.14058 -0.51)
+			(start -0.107836 -0.36)
+			(end 0.107836 -0.36)
 			(stroke
 				(width 0.12)
@@
 		)
 		(fp_line
-			(start -0.14058 0.51)
-			(end 0.14058 0.51)
+			(start -0.107836 0.36)
+			(end 0.107836 0.36)
 			(stroke
 				(width 0.12)
@@
 		)
 		(fp_rect
-			(start -1.48 -0.73)
-			(end 1.48 0.73)
+			(start -0.91 -0.46)
+			(end 0.91 0.46)
 			(stroke
 				(width 0.05)
@@
 		)
 		(fp_rect
-			(start -0.8 -0.4)
-			(end 0.8 0.4)
+			(start -0.5 -0.25)
+			(end 0.5 0.25)
 			(stroke
 				(width 0.1)
@@
 			(effects
 				(font
-					(size 0.4 0.4)
-					(thickness 0.06)
+					(size 0.25 0.25)
+					(thickness 0.04)
 				)
 			)
 		)
 		(pad "1" smd roundrect
-			(at -0.775 0 90)
-			(size 0.9 0.95)
+			(at -0.48 0 90)
+			(size 0.56 0.62)
 			(layers "F.Cu" "F.Mask" "F.Paste")
 			(roundrect_rratio 0.25)
@@
 		)
 		(pad "2" smd roundrect
-			(at 0.775 0 90)
-			(size 0.9 0.95)
+			(at 0.48 0 90)
+			(size 0.56 0.62)
 			(layers "F.Cu" "F.Mask" "F.Paste")
 			(roundrect_rratio 0.25)
@@
 		)
 		(embedded_fonts no)
-		(model "${KICAD10_3DMODEL_DIR}/Capacitor_SMD.3dshapes/C_0603_1608Metric.step"
+		(model "${KICAD10_3DMODEL_DIR}/Capacitor_SMD.3dshapes/C_0402_1005Metric.step"
 			(offset
 				(xyz 0 0 0)
@@
 		(sheetname "/")
 		(sheetfile "Music-player.kicad_sch")
+		(units
+			(unit
+				(name "A")
+				(pins "5" "3" "7" "8" "1" "2" "CD" "6" "G1" "4" "G2" "G3" "G4")
+			)
+		)
 		(attr smd)
 		(duplicate_pad_numbers_are_jumpers no)
@@
 			(property pad_prop_bga)
 			(layers "F.Cu" "F.Mask" "F.Paste")
-			(net "/TPA_EN")
+			(net "unconnected-(U2-NC-PadB12)")
 			(pinfunction "NC_B12")
 			(pintype "no_connect")
@@
 			(net "VDD")
 			(pinfunction "VDD_L1")
-			(pintype "power_in")
+			(pintype "passive")
 		)
 		(pad "L31" smd circle
@@
 		(sheetname "/")
 		(sheetfile "Music-player.kicad_sch")
+		(units
+			(unit
+				(name "A")
+				(pins "2" "1" "3" "4" "5" "6" "7" "8")
+			)
+		)
 		(attr through_hole)
 		(duplicate_pad_numbers_are_jumpers no)
@@
 	)
 	(segment
+		(start 141 82.88)
+		(end 141.465 83.345)
+		(width 0.15)
+		(layer "F.Cu")
+		(net "VDD")
+	)
+	(segment
 		(start 145.95 90.4)
 		(end 145.95 91.27)
@@
 	)
 	(segment
-		(start 144.95 85.3)
-		(end 142.995 83.345)
-		(width 0.15)
-		(layer "F.Cu")
-		(net "VDD")
-	)
-	(segment
 		(start 148.37 89.52)
 		(end 148.35 89.5)
@@
 	)
 	(segment
-		(start 142.995 83.345)
-		(end 141.22 83.345)
-		(width 0.15)
-		(layer "F.Cu")
-		(net "VDD")
-	)
-	(segment
 		(start 144.73 91.3)
 		(end 144.73 90.41)
@@
 	)
 	(segment
+		(start 141.465 83.345)
+		(end 142.995 83.345)
+		(width 0.15)
+		(layer "F.Cu")
+		(net "VDD")
+	)
+	(segment
 		(start 132.25 81.8)
 		(end 135.52 81.8)
@@
 	)
 	(segment
-		(start 141.22 83.345)
-		(end 140.95 83.075)
+		(start 142.995 83.345)
+		(end 144.95 85.3)
 		(width 0.15)
 		(layer "F.Cu")
@@
 	)
 	(via
+		(at 141 82.88)
+		(size 0.5)
+		(drill 0.3)
+		(layers "F.Cu" "B.Cu")
+		(net "VDD")
+	)
+	(via
 		(at 146.4 81.33)
 		(size 0.5)
@@
 	)
 	(via
-		(at 140.95 83.075)
-		(size 0.5)
-		(drill 0.3)
-		(layers "F.Cu" "B.Cu")
-		(net "VDD")
-	)
-	(via
 		(at 156.3 97.48)
 		(size 0.5)
@@
 	)
 	(segment
+		(start 141 81.92)
+		(end 141 81.4)
+		(width 0.15)
+		(layer "F.Cu")
+		(net "GND")
+	)
+	(segment
 		(start 150.93 81.25)
 		(end 150.93 81.24)
@@
 	)
 	(segment
+		(start 141 81.4)
+		(end 141.25 81.15)
+		(width 0.15)
+		(layer "F.Cu")
+		(net "GND")
+	)
+	(segment
 		(start 154.735 100.1)
 		(end 156.46 100.1)
@@
 	)
 	(via
+		(at 141.25 81.15)
+		(size 0.5)
+		(drill 0.3)
+		(layers "F.Cu" "B.Cu")
+		(net "GND")
+	)
+	(via
 		(at 151.95 80.22)
 		(size 0.5)
@@
 		(size 0.5)
 		(drill 0.3)
-		(layers "F.Cu" "B.Cu")
-		(net "GND")
-	)
-	(via
-		(at 140.95 81.525)
-		(size 0.5)
-		(drill 0.3)

Commit message: Add files via upload
Other:
- board text added: "ACE6RINGS NOIR"

Commit message: Add files via upload
Connections:
- U2 pad B12: unconnected-(U2-NC-PadB12) -> /TPA_EN
Changed lines of the file:
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@@
 		(at 125.6 98.25)
 		(property "Reference" "J5"
-			(at 0.775 -2.425 0)
+			(at 6.4 2.9 0)
 			(layer "F.SilkS")
-			(hide yes)
 			(effects
 				(font
-					(size 0.480598 0.480598)
-					(thickness 0.12015)
+					(size 1 1)
 				)
 			)
@@
 		(tags "SOT-143")
 		(property "Reference" "D2"
-			(at 0.02 -5.85 90)
+			(at -2.2 -0.6 180)
 			(layer "F.SilkS")
-			(hide yes)
 			(effects
 				(font
@@
 		(tags "connector JST PH horizontal")
 		(property "Reference" "U1"
-			(at 8 -2.55 0)
+			(at -3.4 1.6 0)
 			(layer "F.SilkS")
-			(hide yes)
 			(effects
 				(font
@@
 		(tags "SOT TO_SOT_SMD")
 		(property "Reference" "U5"
-			(at 0 -2.4 180)
+			(at 1 -2.45 180)
 			(layer "F.SilkS")
-			(hide yes)
 			(effects
 				(font
@@
 		(tags "connector JST PH horizontal")
 		(property "Reference" "J2"
-			(at 2.3125 -3.15 90)
+			(at -3.1 2.6 0)
 			(layer "F.SilkS")
-			(hide yes)
 			(effects
 				(font
@@
 		(tags "NX2016SA-32MHZ-EXS00A-CS06654 ")
 		(property "Reference" "Y2"
-			(at 0 0 0)
+			(at 0.075 -2.3 0)
 			(unlocked yes)
 			(layer "F.SilkS")
-			(hide yes)
 			(effects
 				(font
@@
 		(at 124.5 82.85 -90)
 		(property "Reference" "J4"
-			(at -1.175 -11.135 90)
+			(at 7.95 -9.75 180)
 			(layer "F.SilkS")
-			(hide yes)
 			(effects
 				(font
@@
 			(at 0 -2.4 0)
 			(layer "F.SilkS")
-			(hide yes)
 			(effects
 				(font
@@
 		(tags "USB C Type-C Receptacle SMD USB 2.0 16P 16C USB4105-15-A USB4105-15-A-060 USB4105-15-A-120 USB4105-GF-A USB4105-GF-A-060 USB4105-GF-A-120")
 		(property "Reference" "J1"
-			(at 0 -5.5 270)
+			(at -6 0.01 0)
 			(unlocked yes)
 			(layer "F.SilkS")
-			(hide yes)
 			(effects
 				(font
@@
 		(tags "aqfn qfn nordic nrf nrf5340 aqfn94")
 		(property "Reference" "U2"
-			(at 0 -4.5 0)
+			(at -5.75 4.3 0)
 			(layer "F.SilkS")
-			(hide yes)
 			(effects
 				(font
@@
 			(property pad_prop_bga)
 			(layers "F.Cu" "F.Mask" "F.Paste")
-			(net "unconnected-(U2-NC-PadB12)")
+			(net "/TPA_EN")
 			(pinfunction "NC_B12")
 			(pintype "no_connect")
@@
 			(net "VDD")
 			(pinfunction "VDD_L1")
-			(pintype "passive")
+			(pintype "power_in")
 		)
 		(pad "L31" smd circle
@@
 		(tags "MPZ1608S221ATA00 ")
 		(property "Reference" "FB2"
-			(at 0 0 180)
+			(at 0.5222 1.3 0)
 			(unlocked yes)
 			(layer "F.SilkS")
-			(hide yes)
 			(effects
 				(font
@@
 		(tags "SOT TO_SOT_SMD")
 		(property "Reference" "Q1"
-			(at 0 -2.4 0)
+			(at -0.0125 2.3 0)
 			(layer "F.SilkS")
-			(hide yes)
 			(effects
 				(font
@@
 		(tags "SOT TO_SOT_SMD")
 		(property "Reference" "U3"
-			(at 0 -2.4 180)
+			(at 0 -2.9875 180)
 			(layer "F.SilkS")
-			(hide yes)
 			(effects
 				(font
@@
 		(descr "2012/2, Crystal, 2.0x1.2mm package, SMD, http://txccrystal.com/images/pdf/9ht11.pdf")
 		(property "Reference" "Y1"
-			(at 0 -1.8 90)
+			(at 0.55 -1.7 90)
 			(layer "F.SilkS")
-			(hide yes)
 			(effects
 				(font
@@
 		(tags "TSSOP SO")
 		(property "Reference" "U7"
-			(at 0 -4.2 0)
+			(at 4.7775 1.675 0)
 			(layer "F.SilkS")
-			(hide yes)
 			(effects
 				(font
@@
 		(tags "MPZ1608S221ATA00 ")
 		(property "Reference" "FB1"
-			(at 2.85 0.65 270)
+			(at -0.5 2.05 0)
 			(unlocked yes)
 			(layer "F.SilkS")
-			(hide yes)
 			(effects
 				(font
@@
 		(tags "connector JST PH horizontal")
 		(property "Reference" "U4"
-			(at 7 -2.55 0)
+			(at 17.4 0 0)
 			(layer "F.SilkS")
-			(hide yes)
 			(effects
 				(font
@@
 		(tags "WQFN NoLead")
 		(property "Reference" "U6"
-			(at 0 -2.83 0)
+			(at -2.075 -2.45 0)
 			(layer "F.SilkS")
-			(hide yes)
 			(effects
 				(font
@@
 		(at 167 97.3485 90)
 		(property "Reference" "E1"
-			(at -1.714265 -2.013025 90)
+			(at -0.0515 -2.05 90)
 			(layer "F.SilkS")
-			(hide yes)
 			(effects
 				(font
@@
 		(tags "connector JST PH horizontal")
 		(property "Reference" "J3"
-			(at 1 -2.55 90)
+			(at 5.05 5.55 180)
 			(layer "F.SilkS")
-			(hide yes)
 			(effects
 				(font
@@
 	)
 	(segment
-		(start 156.4 66.782107)
+		(start 156.4 66.7)
 		(end 156.4 65.35)
 		(width 0.2)
@@
 	)
 	(segment
-		(start 141 93.5)
-		(end 140 92.5)
+		(start 143.025 80.107107)
+		(end 143.025 80.075)
 		(width 0.2)
 		(layer "B.Cu")
@@
 	(segment
 		(start 140 92.5)
-		(end 140 83.182107)
+		(end 140 83.1)
 		(width 0.2)
 		(layer "B.Cu")
@@
 	)
 	(segment
-		(start 140 83.182107)
-		(end 156.4 66.782107)
+		(start 140 83.1)
+		(end 141.45 81.65)
 		(width 0.2)
 		(layer "B.Cu")
@@
 	)
 	(segment
-		(start 148.933276 93.5)
-		(end 141 93.5)
+		(start 141.45 81.65)
+		(end 141.457107 81.65)
+		(width 0.2)
+		(layer "B.Cu")
+		(net "/SST_CS")
+	)
+	(segment
+		(start 142.7 80.4)
+		(end 142.732107 80.4)
+		(width 0.2)
+		(layer "B.Cu")
+		(net "/SST_CS")
+	)
+	(segment
+		(start 142.732107 80.4)
+		(end 143.025 80.107107)
+		(width 0.2)
+		(layer "B.Cu")
+		(net "/SST_CS")
+	)
+	(segment
+		(start 141.457107 81.65)
+		(end 141.75 81.357107)
 		(width 0.2)
 		(layer "B.Cu")
@@
 	)
 	(segment
+		(start 141.75 81.35)
+		(end 142.7 80.4)
+		(width 0.2)
+		(layer "B.Cu")
+		(net "/SST_CS")
+	)
+	(segment
+		(start 143.025 80.075)
+		(end 156.4 66.7)
+		(width 0.2)
+		(layer "B.Cu")
+		(net "/SST_CS")
+	)
+	(segment
+		(start 141 93.5)
+		(end 140 92.5)
+		(width 0.2)
+		(layer "B.Cu")
+		(net "/SST_CS")
+	)
+	(segment
+		(start 148.933276 93.5)
+		(end 141 93.5)
+		(width 0.2)
+		(layer "B.Cu")
+		(net "/SST_CS")
+	)
+	(segment
+		(start 141.75 81.357107)
+		(end 141.75 81.35)
+		(width 0.2)
+		(layer "B.Cu")
+		(net "/SST_CS")
+	)
+	(segment
 		(start 150.367834 92.961147)
 		(end 150.367834 92.932166)
@@
 	)
 	(segment
-		(start 154.4 67.317893)
-		(end 139 82.717893)
+		(start 154.4 67.25)
+		(end 149.6 72.05)
 		(width 0.2)
 		(layer "B.Cu")
@@
 	)
 	(segment
-		(start 139 82.717893)
-		(end 139 93)
+		(start 149.6 72.057107)
+		(end 149.307107 72.35)
+		(width 0.2)
+		(layer "B.Cu")
+		(net "/DC")
+	)
+	(segment
+		(start 148.8 94.5)
+		(end 150.338853 92.961147)
+		(width 0.2)
+		(layer "B.Cu")
+		(net "/DC")
+	)
+	(segment
+		(start 149.6 72.05)
+		(end 149.6 72.057107)
+		(width 0.2)
+		(layer "B.Cu")
+		(net "/DC")
+	)
+	(segment
+		(start 150.338853 92.961147)
+		(end 150.367834 92.961147)
 		(width 0.2)
 		(layer "B.Cu")
@@
 	(segment
 		(start 154.4 65.35)
-		(end 154.4 67.317893)
+		(end 154.4 67.25)
 		(width 0.2)
 		(layer "B.Cu")
@@
 	)
 	(segment
-		(start 148.8 94.5)
-		(end 150.338853 92.961147)
+		(start 149.307107 72.35)
+		(end 149.3 72.35)
 		(width 0.2)
 		(layer "B.Cu")
@@
 	)
 	(segment
-		(start 150.338853 92.961147)
-		(end 150.367834 92.961147)
+		(start 149.3 72.35)
+		(end 139 82.65)
+		(width 0.2)
+		(layer "B.Cu")
+		(net "/DC")
+	)
+	(segment
+		(start 139 82.65)
+		(end 139 93)
 		(width 0.2)
 		(layer "B.Cu")
