File: ELECTRONICS/Music-player.kicad_pcb (KiCad board)
At the start: 6 copper layers, 50 x 50 mm, 95 parts, among them J1 USB_C_Receptacle_USB2.0_16P, J2 Screw_Terminal_01x03, J3 Screw_Terminal_01x02, J4 MSD-4-A, J5 SJ-43514, Q1 DMG2301L, Q2 DMG2301L, SW1 RESET, U2 nRF5340-QKxx, U3 SPX3819M5-L-3-3, U5 MCP73831-2-OT, U6 TPA6132A2RTE, U7 PCM5102A, Y1 Seiko SC-20S, Y2 NX2016SA-CS06654

Commit message: Add files via upload
Parts:
- added C9: 4.7u, Capacitor_SMD:C_0603_1608Metric, F.Cu at (147.0, 78.3)
- moved C9 0.25 mm to (144.7, 79.8)
Connections:
- C9 pad 1: Net-(U2-DECUSB) -> Net-(U2-VBUS)
- R4 pad 2: Net-(U2-DECUSB) -> Net-(U2-VBUS)
- U2 pad A5: Net-(U2-DECUSB) -> Net-(U2-VBUS)
- U2 pad B12: /TPA_EN -> unconnected-(U2-NC-PadB12)
Routing:
- net Net-(U2-VBUS): track 0.00 -> 13.3 mm
- net Net-(U2-DECUSB): track 12.7 -> 5.63 mm
- net GND: track 34.5 -> 35.9 mm, vias 62 -> 63
Changed lines of the file:
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@@
 		)
 	)
+	(footprint "Capacitor_SMD:C_0603_1608Metric"
+		(layer "F.Cu")
+		(at 147.025 78.3)
+		(descr "Capacitor SMD 0603 (1608 Metric), square (rectangular) end terminal, IPC-7351 nominal, (Body size source: IPC-SM-782 page 76, https://www.pcb-3d.com/wordpress/wp-content/uploads/ipc-sm-782a_amendment_1_and_2.pdf)")
+		(tags "capacitor")
+		(property "Reference" "C9"
+			(at 1 -0.41 0)
+			(layer "F.SilkS")
+			(hide yes)
+			(effects
+				(font
+					(size 1 1)
+					(thickness 0.15)
+				)
+			)
+		)
+		(property "Value" "4.7u"
+			(at 0 1.43 0)
+			(layer "F.Fab")
+			(effects
+				(font
+					(size 1 1)
+					(thickness 0.15)
+				)
+			)
+		)
+		(property "Datasheet" ""
+			(at 0 0 0)
+			(layer "F.Fab")
+			(hide yes)
+			(effects
+				(font
+					(size 1.27 1.27)
+				)
+			)
+		)
+		(property "Description" "Unpolarized capacitor"
+			(at 0 0 0)
+			(layer "F.Fab")
+			(hide yes)
+			(effects
+				(font
+					(size 1.27 1.27)
+				)
+			)
+		)
+		(property "KiLib_Generator" "SMD_2terminal_chip_molded"
+			(at 0 0 0)
+			(layer "F.SilkS")
+			(hide yes)
+			(effects
+				(font
+					(size 1 1)
+					(thickness 0.15)
+				)
+			)
+		)
+		(property ki_fp_filters "C_*")
+		(sheetname "/")
+		(sheetfile "Music-player.kicad_sch")
+		(attr smd)
+		(duplicate_pad_numbers_are_jumpers no)
+		(fp_line
+			(start -0.14058 -0.51)
+			(end 0.14058 -0.51)
+			(stroke
+				(width 0.12)
+				(type solid)
+			)
+			(layer "F.SilkS")
+		)
+		(fp_line
+			(start -0.14058 0.51)
+			(end 0.14058 0.51)
+			(stroke
+				(width 0.12)
+				(type solid)
+			)
+			(layer "F.SilkS")
+		)
+		(fp_rect
+			(start -1.48 -0.73)
+			(end 1.48 0.73)
+			(stroke
+				(width 0.05)
+				(type solid)
+			)
+			(fill no)
+			(layer "F.CrtYd")
+		)
+		(fp_rect
+			(start -0.8 -0.4)
+			(end 0.8 0.4)
+			(stroke
+				(width 0.1)
+				(type solid)
+			)
+			(fill no)
+			(layer "F.Fab")
+		)
+		(fp_text user "${REFERENCE}"
+			(at 0 0 0)
+			(layer "F.Fab")
+			(effects
+				(font
+					(size 0.4 0.4)
+					(thickness 0.06)
+				)
+			)
+		)
+		(pad "1" smd roundrect
+			(at -0.775 0)
+			(size 0.9 0.95)
+			(layers "F.Cu" "F.Mask" "F.Paste")
+			(roundrect_rratio 0.25)
+			(net "Net-(U2-DECUSB)")
+			(pintype "passive")
+		)
+		(pad "2" smd roundrect
+			(at 0.775 0)
+			(size 0.9 0.95)
+			(layers "F.Cu" "F.Mask" "F.Paste")
+			(roundrect_rratio 0.25)
+			(net "GND")
+			(pintype "passive")
+		)
+		(embedded_fonts no)
+		(model "${KICAD10_3DMODEL_DIR}/Capacitor_SMD.3dshapes/C_0603_1608Metric.step"
+			(offset
+				(xyz 0 0 0)
+			)
+			(scale
+				(xyz 1 1 1)
+			)
+			(rotate
+				(xyz 0 0 0)
+			)
+		)
+	)
 	(footprint "Resistor_SMD:R_0402_1005Metric"
 		(layer "F.Cu")
@@
 	(footprint "Capacitor_SMD:C_0603_1608Metric"
 		(layer "F.Cu")
-		(at 144.9 79.85 90)
+		(at 144.65 79.85 90)
 		(descr "Capacitor SMD 0603 (1608 Metric), square (rectangular) end terminal, IPC-7351 nominal, (Body size source: IPC-SM-782 page 76, https://www.pcb-3d.com/wordpress/wp-content/uploads/ipc-sm-782a_amendment_1_and_2.pdf)")
 		(tags "capacitor")
@@
 			(layers "F.Cu" "F.Mask" "F.Paste")
 			(roundrect_rratio 0.25)
-			(net "Net-(U2-DECUSB)")
+			(net "Net-(U2-VBUS)")
 			(pintype "passive")
 		)
@@
 			(layers "F.Cu" "F.Mask" "F.Paste")
 			(roundrect_rratio 0.25)
-			(net "Net-(U2-DECUSB)")
+			(net "Net-(U2-VBUS)")
 			(pintype "passive")
 		)
@@
 			(property pad_prop_bga)
 			(layers "F.Cu" "F.Mask" "F.Paste")
-			(net "Net-(U2-DECUSB)")
+			(net "Net-(U2-VBUS)")
 			(pinfunction "VBUS_A5")
 			(pintype "power_in")
@@
 			(property pad_prop_bga)
 			(layers "F.Cu" "F.Mask" "F.Paste")
-			(net "/TPA_EN")
+			(net "unconnected-(U2-NC-PadB12)")
 			(pinfunction "NC_B12")
 			(pintype "no_connect")
@@
 			(net "VDD")
 			(pinfunction "VDD_L1")
-			(pintype "power_in")
+			(pintype "passive")
 		)
 		(pad "L31" smd circle
@@
 	)
 	(segment
+		(start 144.65 79.075)
+		(end 144.65 77.8)
+		(width 0.15)
+		(layer "F.Cu")
+		(net "GND")
+	)
+	(segment
 		(start 156.3 103.4)
 		(end 154.785 103.4)
@@
 	)
 	(segment
+		(start 144.65 77.8)
+		(end 144.7 77.75)
+		(width 0.15)
+		(layer "F.Cu")
+		(net "GND")
+	)
+	(segment
 		(start 158 87.35)
 		(end 158 86.255)
@@
 	)
 	(via
+		(at 147.8 78.3)
+		(size 0.5)
+		(drill 0.3)
+		(layers "F.Cu" "B.Cu")
+		(net "GND")
+	)
+	(via
 		(at 148.95 80.24)
 		(size 0.5)
@@
 	)
 	(via
+		(at 144.7 77.75)
+		(size 0.5)
+		(drill 0.3)
+		(layers "F.Cu" "B.Cu")
+		(net "GND")
+	)
+	(via
 		(at 153.85 96.35)
 		(size 0.5)
@@
 	)
 	(via
-		(at 144.9 79.075)
-		(size 0.5)
-		(drill 0.3)
-		(layers "F.Cu" "B.Cu")
-		(net "GND")
-	)
-	(via
 		(at 153 67.8)
 		(size 0.5)
@@
 	)
 	(segment
-		(start 145.725 81.45)
-		(end 145.725 82.325)
-		(width 0.2)
-		(layer "F.Cu")
-		(net "Net-(U2-DECUSB)")
-	)
-	(segment
-		(start 146.64 72.55)
-		(end 146.64 73.41)
-		(width 0.2)
-		(layer "F.Cu")
-		(net "Net-(U2-DECUSB)")
-	)
-	(segment
-		(start 146.64 73.41)
-		(end 145.725 74.325)
-		(width 0.2)
-		(layer "F.Cu")
-		(net "Net-(U2-DECUSB)")
-	)
-	(segment
-		(start 146.15 83.5)
-		(end 146.15 83.3)
-		(width 0.2)
-		(layer "F.Cu")
-		(net "Net-(U2-DECUSB)")
-	)
-	(segment
-		(start 144.9 80.625)
-		(end 145.725 81.45)
-		(width 0.2)
+		(start 145.75 78.8)
+		(end 145.75 81.95)
+		(width 0.15)
 		(layer "F.Cu")
 		(net "Net-(U2-DECUSB)")
 	)
 	(segment
-		(start 145.95 82.55)
-		(end 145.95 83.1)
-		(width 0.2)
+		(start 145.75 81.95)
+		(end 146.225 82.425)
+		(width 0.15)
 		(layer "F.Cu")
 		(net "Net-(U2-DECUSB)")
 	)
 	(segment
-		(start 146.15 83.3)
-		(end 145.95 83.1)
-		(width 0.2)
+		(start 146.25 78.3)
+		(end 145.75 78.8)
+		(width 0.15)
 		(layer "F.Cu")
 		(net "Net-(U2-DECUSB)")
 	)
 	(segment
-		(start 145.725 82.325)
-		(end 145.95 82.55)
-		(width 0.2)
+		(start 146.225 83.425)
+		(end 146.15 83.5)
+		(width 0.15)
 		(layer "F.Cu")
 		(net "Net-(U2-DECUSB)")
 	)
 	(segment
-		(start 145.725 74.325)
-		(end 145.725 81.45)
-		(width 0.2)
+		(start 146.225 82.425)
+		(end 146.225 83.425)
+		(width 0.15)
 		(layer "F.Cu")
 		(net "Net-(U2-DECUSB)")
@@
 		(net "Net-(U6-HPVDD)")
 	)
+	(segment
+		(start 144.65 80.625)
+		(end 144.65 81.25)
+		(width 0.2)
+		(layer "F.Cu")
+		(net "Net-(U2-VBUS)")
+	)
+	(segment
+		(start 145.45 82.05)
+		(end 145.95 82.55)
+		(width 0.2)
+		(layer "F.Cu")
+		(net "Net-(U2-VBUS)")
+	)
+	(segment
+		(start 146.64 72.55)
+		(end 146.64 73.41)
+		(width 0.2)
+		(layer "F.Cu")
+		(net "Net-(U2-VBUS)")
+	)
+	(segment
+		(start 146.64 73.41)
+		(end 145.45 74.6)
+		(width 0.2)
+		(layer "F.Cu")
+		(net "Net-(U2-VBUS)")
+	)
+	(segment
+		(start 145.45 74.6)
+		(end 145.45 82.05)
+		(width 0.2)
+		(layer "F.Cu")
+		(net "Net-(U2-VBUS)")
+	)
+	(segment
+		(start 145.95 82.55)
+		(end 145.95 83.1)
+		(width 0.2)
+		(layer "F.Cu")
+		(net "Net-(U2-VBUS)")
+	)
+	(segment
+		(start 144.65 81.25)
+		(end 145.45 82.05)
+		(width 0.2)
+		(layer "F.Cu")
+		(net "Net-(U2-VBUS)")
+	)
+	(segment
+		(start 144.65 80.625)
+		(end 144.9 80.625)
+		(width 0.2)
+		(layer "F.Cu")
+		(net "Net-(U2-VBUS)")
+	)
 	(zone
