File: ELECTRONICS/Music-player.kicad_sch (KiCad schematic)
At the start: 94 parts, among them J1 USB_C_Receptacle_USB2.0_16P, J2 Screw_Terminal_01x03, J3 Screw_Terminal_01x02, J4 MSD-4-A, J5 SJ-43514, Q1 DMG2301L, Q2 DMG2301L, SW1 RESET, U2 nRF5340-QKxx, U3 SPX3819M5-L-3-3, U5 MCP73831-2-OT, U6 TPA6132A2RTE, U7 PCM5102A, Y1 Seiko SC-20S, Y2 NX2016SA-CS06654

Commit message: Add files via upload
Parts:
- C5: now fitted
Connections:
- net at C9.1, R4.2, U2.A5 (VBUS): no longer C5.1, U2.B6 (DECUSB)
- new net: C5.1, U2.B6 (DECUSB)
Changed lines of the file:
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@@
 	)
 	(junction
-		(at 69.85 224.79)
-		(diameter 0)
-		(color 0 0 0 0)
-	)
-	(junction
 		(at 297.18 237.49)
 		(diameter 0)
@@
 	)
 	(junction
-		(at 76.2 224.79)
-		(diameter 0)
-		(color 0 0 0 0)
-	)
-	(junction
 		(at 222.25 187.96)
 		(diameter 0)
@@
 	(wire
 		(pts
-			(xy 69.85 224.79) (xy 76.2 224.79)
-		)
-		(stroke
-			(width 0)
-			(type default)
-		)
-	)
-	(wire
-		(pts
 			(xy 248.92 26.67) (xy 248.92 24.13)
 		)
@@
 	(wire
 		(pts
-			(xy 69.85 224.79) (xy 69.85 227.33)
+			(xy 69.85 222.25) (xy 69.85 227.33)
 		)
 		(stroke
@@
 	(wire
 		(pts
-			(xy 69.85 222.25) (xy 69.85 224.79)
-		)
-		(stroke
-			(width 0)
-			(type default)
-		)
-	)
-	(wire
-		(pts
 			(xy 209.55 30.48) (xy 209.55 33.02)
 		)
@@
 		(on_board no)
 		(in_pos_files yes)
-		(dnp yes)
+		(dnp no)
 		(property "Reference" "C5"
 			(at 76.454 230.632 0)
